File: teensy4theremin/kicad/sensor/phase_shift_sensor_smd/phase_shift_sensor_smd.kicad_pcb (KiCad board)
At the start: 2 copper layers, 50.2 x 20.3 mm, 20 parts, among them J1 INDUCTOR_IN, J2 INDUCTOR_OUT, J3 ANTENNA, J4 SENSOR, U1 NC7WZ04, U2 IP4220CZ6, U3 REG_3V3

Commit message: update kicad project
Parts:
- removed R1: 22, Resistor_SMD:R_1206_3216Metric_Pad1.42x1.75mm_HandSolder
- added C10: 0.1uF, Capacitor_SMD:C_0805_2012Metric_Pad1.15x1.40mm_HandSolder, F.Cu at (136.5, 97.8)
- added C11: 1uF, Capacitor_SMD:C_0805_2012Metric_Pad1.15x1.40mm_HandSolder, F.Cu at (125.7, 134.6)
- added C12: 1uF, Capacitor_SMD:C_0805_2012Metric_Pad1.15x1.40mm_HandSolder, F.Cu at (134.6, 134.6)
- added C13: 0.1uF, Capacitor_SMD:C_0805_2012Metric_Pad1.15x1.40mm_HandSolder, F.Cu at (142.2, 96.5)
- added C8: 0.1uF, Capacitor_SMD:C_0805_2012Metric_Pad1.15x1.40mm_HandSolder, F.Cu at (113.7, 108.6)
- added C9: 0.1uF, Capacitor_SMD:C_0805_2012Metric_Pad1.15x1.40mm_HandSolder, F.Cu at (127.0, 97.8)
- added U4: 74LVC2G04, Package_TO_SOT_SMD:SOT-23-6, F.Cu at (121.9, 97.8)
- added U5: IP4220CZ6, Package_SO:TSOP-6_1.65x3.05mm_P0.95mm, F.Cu at (132.1, 97.8)
- C1, C2, C3: footprint Capacitor_SMD:C_1206_3216Metric_Pad1.42x1.75mm_HandSolder -> Capacitor_SMD:C_0805_2012Metric_Pad1.15x1.40mm_HandSolder
- C4, C5: value 0.1uF -> 2.2pF; footprint Capacitor_SMD:C_1206_3216Metric_Pad1.42x1.75mm_HandSolder -> Capacitor_SMD:C_0805_2012Metric_Pad1.15x1.40mm_HandSolder
- C6: value 1uF -> 2.2pF; footprint Capacitor_SMD:C_1206_3216Metric_Pad1.42x1.75mm_HandSolder -> Capacitor_SMD:C_0805_2012Metric_Pad1.15x1.40mm_HandSolder
- C7: value 1uF -> 0.1uF; footprint Capacitor_SMD:C_1206_3216Metric_Pad1.42x1.75mm_HandSolder -> Capacitor_SMD:C_0805_2012Metric_Pad1.15x1.40mm_HandSolder
- J1: value INDUCTOR_IN -> SENSOR; footprint Connector_PinHeader_2.54mm:PinHeader_1x01_P2.54mm_Horizontal -> Connector_PinHeader_2.54mm:PinHeader_1x05_P2.54mm_Vertical
- J2: value INDUCTOR_OUT -> INDUCTOR_IN; footprint Connector_PinHeader_2.54mm:PinHeader_1x01_P2.54mm_Horizontal -> Connector_PinHeader_2.54mm:PinHeader_1x01_P2.54mm_Vertical
- J3: value ANTENNA -> INDUCTOR_OUT; footprint Connector_PinHeader_2.54mm:PinHeader_1x01_P2.54mm_Horizontal -> Connector_PinHeader_2.54mm:PinHeader_1x01_P2.54mm_Vertical
- J4: value SENSOR -> ANTENNA; footprint Connector_PinHeader_2.54mm:PinHeader_1x05_P2.54mm_Horizontal -> Connector_PinHeader_2.54mm:PinHeader_1x01_P2.54mm_Vertical
- R2, R3: footprint Resistor_SMD:R_1206_3216Metric_Pad1.42x1.75mm_HandSolder -> Resistor_SMD:R_0805_2012Metric_Pad1.15x1.40mm_HandSolder
- U1: value NC7WZ04 -> 74LVC2G04; footprint Package_TO_SOT_SMD:SOT-363_SC-70-6_Handsoldering -> Package_TO_SOT_SMD:SOT-23-6
- moved J4 65.0 mm to (77.5, 87.0)
- moved C4 56.4 mm to (74.3, 116.2)
- moved C5 55.8 mm to (78.1, 116.2), turned to 90 degrees
- moved C6 52.5 mm to (81.9, 116.2)
- moved C1 46.3 mm to (74.3, 110.7), turned to 90 degrees
- moved C2 41.6 mm to (78.1, 110.7), turned to 270 degrees
- moved J2 36.3 mm to (148.6, 96.5)
- moved C3 34.4 mm to (81.9, 110.7)
- moved R2 31.1 mm to (89.5, 116.2)
- moved R3 29.9 mm to (86.4, 116.2)
- moved TP1 26.9 mm to (142.9, 125.7)
- moved U3 25.4 mm to (130.2, 134.6)
- moved J3 19.0 mm to (120.7, 88.3)
- moved U2 16.5 mm to (110.5, 108.6)
- moved U1 14.8 mm to (121.9, 108.6)
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Connections:
- C2 pad 1: Net-(C2-Pad1) -> Net-(C1-Pad2)
- C2 pad 2: Net-(C1-Pad1) -> Net-(C2-Pad2)
- C3 pad 1: Net-(C3-Pad1) -> Net-(C2-Pad2)
- C3 pad 2: Net-(C2-Pad1) -> Net-(C3-Pad2)
- C4 pad 1: +3V3 -> Net-(C1-Pad1)
- C4 pad 2: GND -> Net-(C4-Pad2)
- C5 pad 1: +3V3 -> Net-(C4-Pad2)
- C5 pad 2: GND -> Net-(C5-Pad2)
- C6 pad 1: +5V -> Net-(C5-Pad2)
- J1 pad 1: Net-(J1-Pad1) -> GND
- J2 pad 1: Net-(C3-Pad1) -> Net-(C13-Pad1)
- J3 pad 1: Net-(C3-Pad1) -> Net-(C1-Pad1)
- J4 pad 1: GND -> Net-(C1-Pad1)
- R2 pad 2: Net-(C1-Pad2) -> Net-(C3-Pad2)
- R3 pad 1: Net-(C1-Pad2) -> Net-(C3-Pad2)
- TP1 pad 1: Net-(C1-Pad2) -> Net-(C3-Pad2)
- U1 pad 1: /REF_CLK -> GND
- U1 pad 3: Net-(C1-Pad2) -> Net-(C3-Pad2)
- U1 pad 6: Net-(R1-Pad1) -> Net-(U1-Pad6)
- U2 pad 1: Net-(C1-Pad2) -> Net-(C3-Pad2)
- U2 pad 6: Net-(R1-Pad1) -> Net-(U2-Pad6)
Routing:
- net GND: track 62.5 -> 0.00 mm, vias 3 -> 0
- net +3V3: track 34.8 -> 0.00 mm, vias 4 -> 0
- net Net-(C1-Pad2): track 31.1 -> 0.00 mm
- net Net-(R1-Pad1): track 26.4 -> 0.00 mm
- net /REF_CLK: track 11.4 -> 0.00 mm
- net +5V: track 10.3 -> 0.00 mm
- net Net-(C3-Pad1): track 9.06 -> 0.00 mm
- net Net-(J1-Pad1): track 8.45 -> 0.00 mm
- net /OUT: track 6.14 -> 0.00 mm
- net Net-(C2-Pad1): track 3.94 -> 0.00 mm
- net Net-(C1-Pad1): track 3.86 -> 0.00 mm
Other:
- board size 50.2 x 20.3 mm -> 79 x 20.3 mm
- board text removed: "*"

Commit message: update sensor PCB
Parts:
- C1, C2, C3: value 2.2pF -> 3.3pF
- C10, C8: value 0.1uF -> 0.22uF
- C4, C5, C6: value 2.2pF -> 10pF
- R2, R3: value 470K -> 330K
- moved R3 44.2 mm to (130.2, 110.5)
- moved R2 41.7 mm to (130.2, 106.7), turned to 270 degrees
- moved C3 41.7 mm to (123.2, 104.8), turned to 0 degrees
- moved C6 41.6 mm to (123.2, 111.1), turned to 0 degrees
- moved C2 41.1 mm to (118.7, 104.8), turned to 0 degrees
- moved C5 41.0 mm to (118.7, 111.1), turned to 0 degrees
- moved C1 40.4 mm to (114.3, 104.8), turned to 0 degrees
- moved J3 40.4 mm to (82.5, 101.6)
- moved C4 40.3 mm to (114.3, 111.1), turned to 0 degrees
- moved C11 35.1 mm to (144.1, 104.8)
- moved U3 31.7 mm to (141.0, 104.8)
- moved C12 30.0 mm to (137.8, 104.8)
- moved TP1 26.7 mm to (126.4, 104.8)
- moved TP6 25.3 mm to (126.4, 111.1)
- moved U2 24.2 mm to (134.6, 109.9)
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Connections:
- U4 pad 3: /REF_CLK -> GND
- U4 pad 4: Net-(C13-Pad2) -> Net-(U4-Pad4)
- U5 pad 1: Net-(C13-Pad2) -> Net-(U5-Pad1)
- U5 pad 4: Net-(U5-Pad4) -> Net-(C13-Pad2)
Routing:
- net GND: track 0.00 -> 92.6 mm, vias 0 -> 2
- net Net-(C1-Pad1): track 0.00 -> 42.8 mm
- net +5V: track 0.00 -> 36.8 mm, vias 0 -> 1
- net +3V3: track 0.00 -> 29.5 mm
- net Net-(C3-Pad2): track 0.00 -> 28.1 mm
- net /REF_CLK: track 0.00 -> 21.5 mm
- net Net-(C13-Pad2): track 0.00 -> 16.7 mm
- net /OUT: track 0.00 -> 4.92 mm
- net Net-(C13-Pad1): track 0.00 -> 3.42 mm
- net Net-(C5-Pad2): track 0.00 -> 2.40 mm
- net Net-(C2-Pad2): track 0.00 -> 2.40 mm
- net Net-(C4-Pad2): track 0.00 -> 2.39 mm
- net Net-(C1-Pad2): track 0.00 -> 2.39 mm
- added copper zone on B.Cu, net GND
- added copper zone on F.Cu, net GND
Other:
- board size 79 x 20.3 mm -> 72.4 x 20.3 mm
- board text added: "ANTENNA"
- board text added: "INDUCTOR_IN"
- board text added: "INDUCTOR_OUT"
- board text added: "IND_IN"
- board text added: "IND_OUT"

Commit message: update
Parts:
- moved J3 2.54 mm to (85.1, 101.6)
- moved J4 2.54 mm to (85.1, 106.7)
Routing:
- net Net-(C1-Pad1): track 42.8 -> 40.2 mm
Other:
- board size 72.4 x 20.3 mm -> 70.5 x 19.7 mm
Changed lines of the file:
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@@
   )
   (module Connector_PinHeader_2.54mm:PinHeader_1x01_P2.54mm_Vertical (layer F.Cu)
-    (at 82.55 106.68)
+    (at 85.09 106.68)
     (descr "Through hole straight pin header, 1x01, 2.54mm pitch, single row")
     (tags "Through hole pin header THT 1x01 2.54mm single row")
@@
   )
   (module Connector_PinHeader_2.54mm:PinHeader_1x01_P2.54mm_Vertical (layer F.Cu)
-    (at 82.55 101.6 180)
+    (at 85.09 101.6 180)
     (descr "Through hole straight pin header, 1x01, 2.54mm pitch, single row")
     (tags "Through hole pin header THT 1x01 2.54mm single row")
@@
       (effects (font (size 1 1) (thickness 0.15)))
     )
-    (fp_text value GND (at 0 1.905 180) (layer B.SilkS)
+    (fp_text value GND (at 0 -1.905 180) (layer B.SilkS)
       (effects (font (size 1 1) (thickness 0.15)) (justify mirror))
     )
@@
       (effects (font (size 1 1) (thickness 0.15)))
     )
-    (fp_text value OUT_NOBUF (at 0 1.55) (layer B.SilkS)
+    (fp_text value OUT_NOBUF (at 0 -1.905) (layer B.SilkS)
       (effects (font (size 1 1) (thickness 0.15)) (justify mirror))
     )
@@
     (effects (font (size 0.7 0.7) (thickness 0.1)) (justify mirror))
   )
-  (gr_text INDUCTOR_OUT (at 88.9 101.6) (layer B.SilkS)
+  (gr_text INDUCTOR_OUT (at 91.44 101.6) (layer B.SilkS)
     (effects (font (size 0.7 0.7) (thickness 0.1)) (justify mirror))
   )
-  (gr_text ANTENNA (at 87.63 106.68) (layer B.SilkS)
+  (gr_text ANTENNA (at 90.17 106.68) (layer B.SilkS)
     (effects (font (size 0.7 0.7) (thickness 0.1)) (justify mirror))
   )
-  (gr_text ANTENNA (at 80.01 106.68 90) (layer F.SilkS)
-    (effects (font (size 0.7 0.7) (thickness 0.1)))
-  )
-  (gr_text IND_OUT (at 80.01 101.6 90) (layer F.SilkS)
+  (gr_text ANTENNA (at 82.55 106.68 90) (layer F.SilkS)
+    (effects (font (size 0.7 0.7) (thickness 0.1)))
+  )
+  (gr_text IND_OUT (at 82.55 101.6 90) (layer F.SilkS)
     (effects (font (size 0.7 0.7) (thickness 0.1)))
   )
@@
     (effects (font (size 0.7 0.7) (thickness 0.1)))
   )
-  (dimension 24.765 (width 0.3) (layer Dwgs.User)
-    (gr_text "24.765 mm" (at 139.3825 125.925) (layer Dwgs.User)
+  (dimension 23.495 (width 0.3) (layer Dwgs.User)
+    (gr_text "23.495 mm" (at 140.0175 125.925) (layer Dwgs.User)
       (effects (font (size 1.5 1.5) (thickness 0.3)))
     )
-    (feature1 (pts (xy 127 116.205) (xy 127 124.411421)))
+    (feature1 (pts (xy 128.27 116.205) (xy 128.27 124.411421)))
     (feature2 (pts (xy 151.765 116.205) (xy 151.765 124.411421)))
-    (crossbar (pts (xy 151.765 123.825) (xy 127 123.825)))
-    (arrow1a (pts (xy 127 123.825) (xy 128.126504 123.238579)))
-    (arrow1b (pts (xy 127 123.825) (xy 128.126504 124.411421)))
+    (crossbar (pts (xy 151.765 123.825) (xy 128.27 123.825)))
+    (arrow1a (pts (xy 128.27 123.825) (xy 129.396504 123.238579)))
+    (arrow1b (pts (xy 128.27 123.825) (xy 129.396504 124.411421)))
     (arrow2a (pts (xy 151.765 123.825) (xy 150.638496 123.238579)))
     (arrow2b (pts (xy 151.765 123.825) (xy 150.638496 124.411421)))
@@
     (effects (font (size 1 1) (thickness 0.2)) (justify mirror))
   )
-  (gr_line (start 79.375 114.3) (end 151.765 114.3) (layer Edge.Cuts) (width 0.2))
+  (gr_line (start 81.28 113.665) (end 151.765 113.665) (layer Edge.Cuts) (width 0.2))
   (gr_text GND (at 151.13 105.41 90) (layer F.SilkS)
     (effects (font (size 0.7 0.7) (thickness 0.1)))
@@
     (effects (font (size 0.7 0.7) (thickness 0.1)))
   )
-  (gr_circle (center 81.915 96.52) (end 83.015 96.52) (layer Edge.Cuts) (width 0.15))
-  (gr_circle (center 81.915 111.76) (end 83.015 111.76) (layer Edge.Cuts) (width 0.15))
-  (gr_line (start 79.375 93.98) (end 79.375 114.3) (layer Edge.Cuts) (width 0.2))
-  (gr_line (start 151.765 93.98) (end 151.765 114.3) (layer Edge.Cuts) (width 0.2))
-  (gr_line (start 79.375 93.98) (end 151.765 93.98) (layer Edge.Cuts) (width 0.2))
-  (dimension 72.39 (width 0.3) (layer Dwgs.User)
-    (gr_text "72.390 mm" (at 115.57 81.72) (layer Dwgs.User)
+  (gr_circle (center 84.455 96.52) (end 85.555 96.52) (layer Edge.Cuts) (width 0.15))
+  (gr_circle (center 84.455 111.76) (end 85.555 111.76) (layer Edge.Cuts) (width 0.15))
+  (gr_line (start 81.28 93.98) (end 81.28 113.665) (layer Edge.Cuts) (width 0.2))
+  (gr_line (start 151.765 93.98) (end 151.765 113.665) (layer Edge.Cuts) (width 0.2))
+  (gr_line (start 81.28 93.98) (end 151.765 93.98) (layer Edge.Cuts) (width 0.2))
+  (dimension 70.485 (width 0.3) (layer Dwgs.User)
+    (gr_text "70.485 mm" (at 116.5225 81.72) (layer Dwgs.User)
       (effects (font (size 1.5 1.5) (thickness 0.3)))
     )
     (feature1 (pts (xy 151.765 91.44) (xy 151.765 83.233579)))
-    (feature2 (pts (xy 79.375 91.44) (xy 79.375 83.233579)))
-    (crossbar (pts (xy 79.375 83.82) (xy 151.765 83.82)))
+    (feature2 (pts (xy 81.28 91.44) (xy 81.28 83.233579)))
+    (crossbar (pts (xy 81.28 83.82) (xy 151.765 83.82)))
     (arrow1a (pts (xy 151.765 83.82) (xy 150.638496 84.406421)))
     (arrow1b (pts (xy 151.765 83.82) (xy 150.638496 83.233579)))
-    (arrow2a (pts (xy 79.375 83.82) (xy 80.501504 84.406421)))
-    (arrow2b (pts (xy 79.375 83.82) (xy 80.501504 83.233579)))
-  )
-  (dimension 20.32 (width 0.3) (layer Dwgs.User)
-    (gr_text "20.320 mm" (at 164.612152 104.14 270) (layer Dwgs.User)
+    (arrow2a (pts (xy 81.28 83.82) (xy 82.406504 84.406421)))
+    (arrow2b (pts (xy 81.28 83.82) (xy 82.406504 83.233579)))
+  )
+  (dimension 19.685 (width 0.3) (layer Dwgs.User)
+    (gr_text "19.685 mm" (at 164.66 103.8225 270) (layer Dwgs.User)
       (effects (font (size 1.5 1.5) (thickness 0.3)))
     )
-    (feature1 (pts (xy 154.892152 114.3) (xy 163.098573 114.3)))
-    (feature2 (pts (xy 154.892152 93.98) (xy 163.098573 93.98)))
-    (crossbar (pts (xy 162.512152 93.98) (xy 162.512152 114.3)))
-    (arrow1a (pts (xy 162.512152 114.3) (xy 161.925731 113.173496)))
-    (arrow1b (pts (xy 162.512152 114.3) (xy 163.098573 113.173496)))
-    (arrow2a (pts (xy 162.512152 93.98) (xy 161.925731 95.106504)))
-    (arrow2b (pts (xy 162.512152 93.98) (xy 163.098573 95.106504)))
+    (feature1 (pts (xy 154.94 113.665) (xy 163.146421 113.665)))
+    (feature2 (pts (xy 154.94 93.98) (xy 163.146421 93.98)))
+    (crossbar (pts (xy 162.56 93.98) (xy 162.56 113.665)))
+    (arrow1a (pts (xy 162.56 113.665) (xy 161.973579 112.538496)))
+    (arrow1b (pts (xy 162.56 113.665) (xy 163.146421 112.538496)))
+    (arrow2a (pts (xy 162.56 93.98) (xy 161.973579 95.106504)))
+    (arrow2b (pts (xy 162.56 93.98) (xy 163.146421 95.106504)))
   )
   (segment (start 139.97 104.775) (end 139.97 104.41) (width 0.4) (layer F.Cu) (net 1))
@@
   (segment (start 111.76 109.61) (end 111.76 104.775) (width 0.25) (layer F.Cu) (net 5))
   (segment (start 111.76 104.775) (end 113.275 104.775) (width 0.25) (layer F.Cu) (net 5))
-  (segment (start 111.76 104.775) (end 82.55 104.775) (width 0.25) (layer F.Cu) (net 5))
-  (segment (start 82.55 101.6) (end 82.55 104.775) (width 0.25) (layer F.Cu) (net 5))
-  (segment (start 82.55 104.775) (end 82.55 106.68) (width 0.25) (layer F.Cu) (net 5))
+  (segment (start 85.09 101.6) (end 85.09 104.775) (width 0.25) (layer F.Cu) (net 5))
+  (segment (start 85.09 104.775) (end 85.09 106.68) (width 0.25) (layer F.Cu) (net 5))
+  (segment (start 111.76 104.775) (end 85.09 104.775) (width 0.25) (layer F.Cu) (net 5))
   (segment (start 115.325 104.775) (end 117.72 104.775) (width 0.25) (layer F.Cu) (net 6))
   (segment (start 147.387919 107.95) (end 148.59 107.95) (width 0.25) (layer F.Cu) (net 7))
@@
     (polygon
       (pts
-        (xy 128.27 94.615) (xy 151.13 94.615) (xy 151.13 113.665) (xy 128.27 113.665)
+        (xy 128.27 94.615) (xy 151.13 94.615) (xy 151.13 113.03) (xy 128.27 113.03)
       )
     )
@@
     (polygon
       (pts
-        (xy 128.27 94.615) (xy 151.13 94.615) (xy 151.13 113.665) (xy 128.27 113.665)
+        (xy 128.27 94.615) (xy 151.13 94.615) (xy 151.13 113.03) (xy 128.27 113.03)
       )
     )

Commit message: update sensor pcb - 3v3 regulator
Parts:
- U3: value REG_3V3 -> MCP1700-3302E_SOT23
Connections:
- U3 pad 2: +5V -> +3V3
- U3 pad 3: +3V3 -> +5V
Routing:
- net +5V: track 36.8 -> 39.3 mm
- net +3V3: track 29.5 -> 30.9 mm
Other:
- board size 70.5 x 19.7 mm -> 70.5 x 19.8 mm
- board text added: "Recommended parts: BUFFERS: SN74LVC2G04DBVR x2 ESD: IP4220CZ6 x2 3V3 REG: MCP1700T-3302E x1"
Changed lines of the file:
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@@
   (general
     (thickness 1.6)
-    (drawings 26)
-    (tracks 150)
+    (drawings 29)
+    (tracks 152)
     (zones 0)
     (modules 27)
@@
       (effects (font (size 1 1) (thickness 0.15)))
     )
-    (fp_text value REG_3V3 (at 0 2.5 180) (layer F.Fab)
+    (fp_text value MCP1700-3302E_SOT23 (at 0 2.5 180) (layer F.Fab)
       (effects (font (size 1 1) (thickness 0.15)))
     )
@@
       (net 2 GND))
     (pad 2 smd rect (at -1 0.95 180) (size 0.9 0.8) (layers F.Cu F.Paste F.Mask)
+      (net 1 +3V3))
+    (pad 3 smd rect (at 1 0 180) (size 0.9 0.8) (layers F.Cu F.Paste F.Mask)
       (net 4 +5V))
-    (pad 3 smd rect (at 1 0 180) (size 0.9 0.8) (layers F.Cu F.Paste F.Mask)
-      (net 1 +3V3))
     (model ${KISYS3DMOD}/Package_TO_SOT_SMD.3dshapes/SOT-23.wrl
       (at (xyz 0 0 0))
@@
     )
   )
+  (gr_circle (center 109.22 111.125) (end 110.32 111.125) (layer Edge.Cuts) (width 0.15))
+  (gr_text "Recommended parts:\nBUFFERS: SN74LVC2G04DBVR x2\nESD: IP4220CZ6 x2\n3V3 REG: MCP1700T-3302E x1" (at 116.205 98.425) (layer B.SilkS)
+    (effects (font (size 0.7 0.7) (thickness 0.1)) (justify left mirror))
+  )
+  (gr_circle (center 124.63 96.52) (end 125.73 96.52) (layer Edge.Cuts) (width 0.15))
   (gr_text INDUCTOR_IN (at 143.51 96.52) (layer B.SilkS)
     (effects (font (size 0.7 0.7) (thickness 0.1)) (justify mirror))
@@
     (effects (font (size 1 1) (thickness 0.2)) (justify mirror))
   )
-  (gr_line (start 81.28 113.665) (end 151.765 113.665) (layer Edge.Cuts) (width 0.2))
+  (gr_line (start 81.28 113.792) (end 151.765 113.792) (layer Edge.Cuts) (width 0.2))
   (gr_text GND (at 151.13 105.41 90) (layer F.SilkS)
     (effects (font (size 0.7 0.7) (thickness 0.1)))
@@
     (effects (font (size 0.7 0.7) (thickness 0.1)))
   )
-  (gr_circle (center 84.455 96.52) (end 85.555 96.52) (layer Edge.Cuts) (width 0.15))
-  (gr_circle (center 84.455 111.76) (end 85.555 111.76) (layer Edge.Cuts) (width 0.15))
-  (gr_line (start 81.28 93.98) (end 81.28 113.665) (layer Edge.Cuts) (width 0.2))
-  (gr_line (start 151.765 93.98) (end 151.765 113.665) (layer Edge.Cuts) (width 0.2))
+  (gr_circle (center 83.82 96.52) (end 84.92 96.52) (layer Edge.Cuts) (width 0.15))
+  (gr_circle (center 83.82 111.125) (end 84.92 111.125) (layer Edge.Cuts) (width 0.15))
+  (gr_line (start 81.28 93.98) (end 81.28 113.792) (layer Edge.Cuts) (width 0.2))
+  (gr_line (start 151.765 93.98) (end 151.765 113.792) (layer Edge.Cuts) (width 0.2))
   (gr_line (start 81.28 93.98) (end 151.765 93.98) (layer Edge.Cuts) (width 0.2))
   (dimension 70.485 (width 0.3) (layer Dwgs.User)
@@
     (arrow2b (pts (xy 81.28 83.82) (xy 82.406504 83.233579)))
   )
-  (dimension 19.685 (width 0.3) (layer Dwgs.User)
-    (gr_text "19.685 mm" (at 164.66 103.8225 270) (layer Dwgs.User)
+  (dimension 19.812 (width 0.3) (layer Dwgs.User)
+    (gr_text "19.812 mm" (at 164.66 103.886 270) (layer Dwgs.User)
       (effects (font (size 1.5 1.5) (thickness 0.3)))
     )
-    (feature1 (pts (xy 154.94 113.665) (xy 163.146421 113.665)))
+    (feature1 (pts (xy 154.94 113.792) (xy 163.146421 113.792)))
     (feature2 (pts (xy 154.94 93.98) (xy 163.146421 93.98)))
-    (crossbar (pts (xy 162.56 93.98) (xy 162.56 113.665)))
-    (arrow1a (pts (xy 162.56 113.665) (xy 161.973579 112.538496)))
-    (arrow1b (pts (xy 162.56 113.665) (xy 163.146421 112.538496)))
+    (crossbar (pts (xy 162.56 93.98) (xy 162.56 113.792)))
+    (arrow1a (pts (xy 162.56 113.792) (xy 161.973579 112.665496)))
+    (arrow1b (pts (xy 162.56 113.792) (xy 163.146421 112.665496)))
     (arrow2a (pts (xy 162.56 93.98) (xy 161.973579 95.106504)))
     (arrow2b (pts (xy 162.56 93.98) (xy 163.146421 95.106504)))
   )
-  (segment (start 139.97 104.775) (end 139.97 104.41) (width 0.4) (layer F.Cu) (net 1))
   (segment (start 139.31 103.75) (end 137.795 103.75) (width 0.4) (layer F.Cu) (net 1))
-  (segment (start 139.97 104.41) (end 139.31 103.75) (width 0.4) (layer F.Cu) (net 1))
+  (segment (start 141.97 103.825) (end 141.27 103.825) (width 0.4) (layer F.Cu) (net 1))
+  (segment (start 141.27 103.825) (end 141.195 103.75) (width 0.4) (layer F.Cu) (net 1))
+  (segment (start 141.195 103.75) (end 139.31 103.75) (width 0.4) (layer F.Cu) (net 1))
   (segment (start 134.23 103.75) (end 133.985 103.505) (width 0.4) (layer F.Cu) (net 1))
   (segment (start 142.875 107.315) (end 143.51 107.95) (width 0.4) (layer F.Cu) (net 1))
@@
   (segment (start 133.35 95.25) (end 135.89 95.25) (width 0.25) (layer F.Cu) (net 4))
   (segment (start 144.07 103.825) (end 144.145 103.75) (width 0.25) (layer F.Cu) (net 4))
-  (segment (start 141.97 103.825) (end 144.07 103.825) (width 0.25) (layer F.Cu) (net 4))
   (segment (start 147.32 99.06) (end 148.59 100.33) (width 0.25) (layer F.Cu) (net 4))
   (segment (start 142.875 99.06) (end 147.32 99.06) (width 0.25) (layer F.Cu) (net 4))
@@
   (via (at 144.780002 102.235) (size 0.8) (drill 0.4) (layers F.Cu B.Cu) (net 4))
   (segment (start 144.145 103.75) (end 144.145 102.870002) (width 0.25) (layer F.Cu) (net 4))
+  (segment (start 143.12 104.775) (end 144.145 103.75) (width 0.25) (layer F.Cu) (net 4))
+  (segment (start 139.97 104.775) (end 143.12 104.775) (width 0.25) (layer F.Cu) (net 4))
   (segment (start 113.275 111.125) (end 111.76 109.61) (width 0.25) (layer F.Cu) (net 5))
   (segment (start 111.76 109.61) (end 111.76 104.775) (width 0.25) (layer F.Cu) (net 5))
