File: teensy4theremin/kicad/sensor/analog_switch_heterodyne/analog_switch_heterodyne.kicad_pcb (KiCad board)
At the start: 2 copper layers, 70.5 x 20.1 mm, 15 parts, among them J1 OSC, J2 INDUCTOR_IN, J3 INDUCTOR_OUT, J4 ANTENNA, U1 2G04, U2 4220CZ6

Commit message: update pcb
Parts:
- added C10: 0.1uF, Capacitor_SMD:C_0805_2012Metric_Pad1.15x1.40mm_HandSolder, F.Cu at (122.3, 56.8)
- added C11: 1uF, Capacitor_SMD:C_0805_2012Metric_Pad1.15x1.40mm_HandSolder, F.Cu at (105.4, 69.1)
- added C12: 0.1uF, Capacitor_SMD:C_0805_2012Metric_Pad1.15x1.40mm_HandSolder, F.Cu at (109.2, 69.1)
- added C13: 1uF, Capacitor_SMD:C_0805_2012Metric_Pad1.15x1.40mm_HandSolder, F.Cu at (122.3, 58.7)
- added C14: 0.1uF, Capacitor_SMD:C_0805_2012Metric_Pad1.15x1.40mm_HandSolder, F.Cu at (111.2, 67.1)
- added C15: 1uF, Capacitor_SMD:C_0805_2012Metric_Pad1.15x1.40mm_HandSolder, F.Cu at (122.3, 60.7)
- added C16: 0.1uF, Capacitor_SMD:C_0805_2012Metric_Pad1.15x1.40mm_HandSolder, F.Cu at (126.0, 56.8)
- added C17: 2.2uF, Capacitor_SMD:C_0805_2012Metric_Pad1.15x1.40mm_HandSolder, F.Cu at (118.5, 61.5)
- added C7: 100pF, Capacitor_SMD:C_0805_2012Metric_Pad1.15x1.40mm_HandSolder, F.Cu at (118.5, 59.5)
- added C8: 100pF, Capacitor_SMD:C_0805_2012Metric_Pad1.15x1.40mm_HandSolder, F.Cu at (107.4, 67.1)
- added C9: 1uF, Capacitor_SMD:C_0805_2012Metric_Pad1.15x1.40mm_HandSolder, F.Cu at (101.7, 69.0)
- added L1: Ferrite 10uH, Inductor_SMD:L_1210_3225Metric_Pad1.42x2.65mm_HandSolder, F.Cu at (99.6, 52.7)
- added L2: Ferrite 10uH, Inductor_SMD:L_1210_3225Metric_Pad1.42x2.65mm_HandSolder, F.Cu at (99.6, 49.5)
- added L3: Ferrite 10uH, Inductor_SMD:L_1210_3225Metric_Pad1.42x2.65mm_HandSolder, F.Cu at (107.6, 46.4)
- added L4: Ferrite 10uH, Inductor_SMD:L_1210_3225Metric_Pad1.42x2.65mm_HandSolder, F.Cu at (99.6, 46.3)
- added R4: 10, Resistor_SMD:R_0805_2012Metric_Pad1.15x1.40mm_HandSolder, F.Cu at (119.7, 54.8)
- added R5: 10K, Resistor_SMD:R_0805_2012Metric_Pad1.15x1.40mm_HandSolder, F.Cu at (114.8, 59.5)
- added R6: 22K, Resistor_SMD:R_0805_2012Metric_Pad1.15x1.40mm_HandSolder, F.Cu at (87.7, 69.2)
- C1: value 2.2uF -> 220pF
- C2: value 0.1uF -> 100pF
- C3: value 0.22uF -> 100pF
- C4, C6: value 3.3pF -> 100pF
- C5: value 3.3pF -> 220pF
- J1: value OSC -> SENSOR1; footprint Connector_PinHeader_2.54mm:PinHeader_1x03_P2.54mm_Horizontal -> Connector_PinHeader_2.54mm:PinHeader_1x05_P2.54mm_Vertical
- J2: value INDUCTOR_IN -> OSC1; footprint Connector_PinHeader_2.54mm:PinHeader_1x01_P2.54mm_Vertical -> Connector_PinHeader_2.54mm:PinHeader_1x03_P2.54mm_Horizontal
- J3: value INDUCTOR_OUT -> SENSOR2; footprint Connector_PinHeader_2.54mm:PinHeader_1x01_P2.54mm_Vertical -> Connector_PinHeader_2.54mm:PinHeader_1x05_P2.54mm_Vertical
- J4: value ANTENNA -> OSC2; footprint Connector_PinHeader_2.54mm:PinHeader_1x01_P2.54mm_Horizontal -> Connector_PinHeader_2.54mm:PinHeader_1x03_P2.54mm_Horizontal
- R1: value 2.7M -> 10
- R2: value 10 -> 10K
- R3: value 10 -> 22K
- U1: value 2G04 -> ADG721BRMZ; footprint Package_TO_SOT_SMD:SOT-23-6 -> Package_SO:MSOP-8_3x3mm_P0.65mm
- U2: value 4220CZ6 -> 2G04; footprint Package_SO:TSOP-6_1.65x3.05mm_P0.95mm -> Package_TO_SOT_SMD:SOT-23-6
- moved J1 93.7 mm to (85.1, 31.5)
- moved J3 88.3 mm to (141.5, 32.1), turned to 0 degrees
- moved J4 70.9 mm to (148.6, 71.4), turned to 0 degrees
- moved U1 70.2 mm to (89.9, 59.4), turned to 0 degrees
- moved R3 61.1 mm to (114.8, 57.6), turned to 0 degrees
- moved R1 60.3 mm to (124.7, 48.0), turned to 0 degrees
- moved U2 59.9 mm to (98.4, 59.2), turned to 0 degrees
- moved C2 58.4 mm to (94.2, 69.0), turned to 0 degrees
- moved C6 57.6 mm to (123.5, 54.8), turned to 0 degrees
- moved C5 54.9 mm to (118.5, 57.6), turned to 0 degrees
- moved C3 54.6 mm to (123.6, 51.2), turned to 0 degrees
- moved R2 53.2 mm to (97.9, 69.0), turned to 0 degrees
- moved C1 51.4 mm to (112.9, 69.1), turned to 0 degrees
- moved C4 44.3 mm to (114.8, 61.5)
- moved J2 41.4 mm to (148.3, 56.4)
Connections:
- C1 pad 1: +3V3 -> /OSC1
- C2 pad 1: +3V3 -> Net-(C2-Pad1)
- C3 pad 1: +3V3 -> Net-(C3-Pad1)
- C4 pad 1: GND -> Net-(C4-Pad1)
- C4 pad 2: Net-(C4-Pad2) -> GND
- C5 pad 1: Net-(C5-Pad1) -> /OSC1
- C5 pad 2: Net-(C5-Pad2) -> GND
- C6 pad 1: GND -> Net-(C6-Pad1)
- C6 pad 2: Net-(C5-Pad1) -> GND
- J1 pad 2: /OSC_OUT -> /FREF1
- J1 pad 3: /3.3V -> GND
- J2 pad 1: Net-(C4-Pad2) -> /3.3V_1
- J3 pad 1: Net-(C5-Pad2) -> GND
- J4 pad 1: Net-(C5-Pad2) -> /3.3V_1
- R1 pad 1: Net-(R1-Pad1) -> Net-(C2-Pad1)
- R1 pad 2: Net-(C5-Pad2) -> Net-(R1-Pad2)
- R2 pad 1: Net-(C4-Pad2) -> Net-(C3-Pad1)
- R2 pad 2: Net-(R2-Pad2) -> Net-(C2-Pad1)
- R3 pad 1: /3.3V -> Net-(C4-Pad1)
- R3 pad 2: +3V3 -> Net-(C3-Pad1)
- U1 pad 1: Net-(R1-Pad1) -> /OSC1
- U1 pad 2: GND -> Net-(R1-Pad2)
- U1 pad 3: Net-(R2-Pad2) -> /FREF2
- U1 pad 4: /OSC_OUT -> GND
- U1 pad 5: +3V3 -> /OSC1
- U1 pad 6: Net-(R2-Pad2) -> Net-(R4-Pad2)
- U2 pad 1: Net-(R1-Pad1) -> Net-(C8-Pad1)
- U2 pad 3: Net-(U2-Pad3) -> Net-(C4-Pad1)
- U2 pad 4: Net-(R2-Pad2) -> /HOUT1
- U2 pad 5: +3V3 -> Net-(C15-Pad1)
- U2 pad 6: Net-(U2-Pad6) -> /HOUT2
Routing:
- net GND: track 91.7 -> 0.00 mm, vias 6 -> 0
- net Net-(C5-Pad2): track 52.7 -> 0.00 mm
- net +3V3: track 29.7 -> 0.00 mm, vias 3 -> 0
- net Net-(R2-Pad2): track 15.8 -> 0.00 mm
- net Net-(R1-Pad1): track 14.4 -> 0.00 mm
- net Net-(C4-Pad2): track 8.18 -> 0.00 mm
- net /OSC_OUT: track 3.05 -> 0.00 mm
- net Net-(C5-Pad1): track 3.03 -> 0.00 mm
- net /3.3V: track 2.92 -> 0.00 mm
- removed copper zone on B.Cu, net GND
Other:
- board size 70.5 x 20.1 mm -> 82.8 x 41.3 mm
- board text removed: "(c) Vadim Lopatin, 2020"
- board text removed: "+3.3"
- board text removed: "3.3V"
- board text removed: "ANTENNA"
- board text removed: "GND"
- board text removed: "INDUCTOR_IN"
- board text removed: "INDUCTOR_OUT"
- board text removed: "IND_IN"
- board text removed: "IND_OUT"
- board text removed: "OUT"
- board text removed: "Theremin Oscillator - rev 0.1"
- board text removed: "for Teensy 4 Theremin Project"

Commit message: heterodyne pcb
Parts:
- J1: value SENSOR1 -> H_OUT
- J2: value OSC1 -> OSC_PITCH
- J3: value SENSOR2 -> F_REF
- J4: value OSC2 -> OSC_VOL
- moved L1 50.9 mm to (150.5, 51.4), turned to 270 degrees
- moved J1 50.7 mm to (134.6, 42.5), turned to 90 degrees
- moved C9 50.1 mm to (150.5, 57.8)
- moved U1 50.1 mm to (139.7, 64.8)
- moved R2 49.6 mm to (146.1, 57.1), turned to 270 degrees
- moved C2 49.1 mm to (142.2, 59.1), turned to 180 degrees
- moved R6 48.3 mm to (133.3, 53.3), turned to 270 degrees
- moved J3 45.5 mm to (144.8, 77.5), turned to 270 degrees
- moved L3 43.6 mm to (141.6, 73.7), turned to 180 degrees
- moved U2 43.1 mm to (139.7, 47.0), turned to 90 degrees
- moved C1 37.0 mm to (149.2, 76.2), turned to 270 degrees
- moved L4 33.7 mm to (133.3, 47.6), turned to 90 degrees
- moved C8 33.6 mm to (137.2, 51.4)
- moved C17 31.7 mm to (146.7, 47.0), turned to 90 degrees
- moved R3 31.5 mm to (146.1, 53.3), turned to 270 degrees
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Connections:
- net /HOUT1 renamed /HOUT_PITCH
- C1 pad 1: /OSC1 -> /OSC_PITCH
- C11 pad 1: /3.3V_1 -> /3.3V_2
- C12 pad 1: /3.3V_1 -> /3.3V_2
- C5 pad 1: /OSC1 -> /OSC_VOL
- J1 pad 1: GND -> +3V3
- J1 pad 2: /FREF1 -> /HOUT_VOL
- J1 pad 5: +3V3 -> GND
- J2 pad 2: /OSC1 -> /OSC_PITCH
- J3 pad 1: GND -> +3V3
- J3 pad 2: /FREF2 -> /FREF_VOL
- J3 pad 4: /HOUT2 -> /FREF_PITCH
- J3 pad 5: +3V3 -> GND
- J4 pad 1: /3.3V_1 -> /3.3V_2
- J4 pad 2: /OSC1 -> /OSC_VOL
- L2 pad 2: /3.3V_1 -> /3.3V_2
- U1 pad 1: /OSC1 -> /OSC_VOL
- U1 pad 2: Net-(R1-Pad2) -> Net-(R4-Pad2)
- U1 pad 3: /FREF2 -> /FREF_PITCH
- U1 pad 5: /OSC1 -> /OSC_PITCH
- U1 pad 6: Net-(R4-Pad2) -> Net-(R1-Pad2)
- U1 pad 7: /FREF1 -> /FREF_VOL
- U2 pad 6: /HOUT2 -> /HOUT_VOL
Routing:
- net GND: track 0.00 -> 34.3 mm
- net /FREF_PITCH: track 0.00 -> 9.24 mm
- net Net-(R4-Pad2): track 0.00 -> 9.04 mm
- net Net-(C4-Pad1): track 0.00 -> 8.84 mm
- net Net-(C8-Pad1): track 0.00 -> 8.84 mm
- net Net-(C15-Pad1): track 0.00 -> 8.20 mm
- net Net-(C13-Pad1): track 0.00 -> 8.02 mm
- net /OSC_VOL: track 0.00 -> 7.25 mm
- net /OSC_PITCH: track 0.00 -> 6.07 mm
- net Net-(R1-Pad2): track 0.00 -> 5.44 mm
- net /FREF_VOL: track 0.00 -> 4.63 mm
- net Net-(C2-Pad1): track 0.00 -> 4.55 mm
- net Net-(C3-Pad1): track 0.00 -> 4.55 mm
- net Net-(C6-Pad1): track 0.00 -> 4.55 mm
- net Net-(C7-Pad1): track 0.00 -> 4.54 mm
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Other:
- board size 82.8 x 41.3 mm -> 81.3 x 87 mm

Commit message: analog switch heterodyne PCB and gerber
Parts:
- removed C1, C5: 220pF, Capacitor_SMD:C_0805_2012Metric_Pad1.15x1.40mm_HandSolder
- added L5: Ferrite 10uH, Inductor_SMD:L_1210_3225Metric_Pad1.42x2.65mm_HandSolder, F.Cu at (128.1, 55.2)
- added TP1: PITCH_FLT, TestPoint:TestPoint_Pad_1.0x1.0mm, F.Cu at (146.8, 50.3)
- added TP2: VOL_FLT, TestPoint:TestPoint_Pad_1.0x1.0mm, F.Cu at (132.6, 50.3)
- added U3: 2G04, Package_TO_SOT_SMD:SOT-23-6, F.Cu at (139.7, 72.3)
- C12: value 0.1uF -> 1uF
- R1, R4: value 10 -> 100
- R2, R5: value 10K -> 4.7K
- R3, R6: value 22K -> 47K
- moved L3 20.8 mm to (151.3, 55.2)
- moved C12 13.3 mm to (136.9, 72.3), turned to 270 degrees
- moved C10 13.3 mm to (142.6, 72.3), turned to 270 degrees
- moved L1 8.93 mm to (151.3, 60.3), turned to 180 degrees
- moved L2 8.93 mm to (128.1, 60.3), turned to 0 degrees
- moved C11 7.33 mm to (130.0, 64.4), turned to 0 degrees
- moved C9 7.08 mm to (149.4, 64.8)
- moved L4 5.87 mm to (128.1, 50.2), turned to 0 degrees
- moved C17 5.34 mm to (150.9, 50.3), turned to 180 degrees
- moved J2 2.84 mm to (147.3, 68.6)
- moved J4 2.84 mm to (132.1, 73.7)
- moved C13 1.27 mm to (139.7, 69.2)
- moved J3 1.27 mm to (144.8, 78.7)
- moved C14 0.76 mm to (139.7, 67.2)
- moved C3 0.64 mm to (142.2, 55.9)
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Connections:
- net Net-(C13-Pad1) renamed /VCC_U1
- net Net-(C15-Pad1) renamed /VCC_U2
- C10 pad 1: /3.3V_1 -> /VCC_U3
- C12 pad 1: /3.3V_2 -> /VCC_U3
- U1 pad 1: /OSC_VOL -> Net-(U1-Pad1)
- U1 pad 5: /OSC_PITCH -> Net-(U1-Pad5)
Routing:
- net +3V3: track 0.00 -> 122.5 mm
- net GND: track 34.3 -> 137.2 mm, vias 0 -> 6
- net /VCC_U3: track 0.00 -> 26.5 mm
- net /VCC_U1: track 8.02 -> 24.0 mm, vias 0 -> 3
- net /3.3V_2: track 0.00 -> 15.5 mm
- net /FREF_VOL: track 4.63 -> 17.7 mm, vias 0 -> 1
- net Net-(U1-Pad1): track 0.00 -> 9.88 mm
- net /3.3V_1: track 0.00 -> 9.51 mm
- net /VCC_U2: track 8.20 -> 17.7 mm
- net /FREF_PITCH: track 9.24 -> 16.5 mm, vias 0 -> 1
- net Net-(U1-Pad5): track 0.00 -> 7.17 mm
- net Net-(R4-Pad2): track 9.04 -> 4.64 mm
- net Net-(C4-Pad1): track 8.84 -> 11.1 mm
- net Net-(C8-Pad1): track 8.84 -> 11.1 mm
- net /OSC_PITCH: track 6.07 -> 7.60 mm
- added copper zone on B.Cu, net GND
Other:
- board size 81.3 x 87 mm -> 30.5 x 40.6 mm
- board text added: "+3.3"
- board text added: "+3.3_P"
- board text added: "+3.3_V"
- board text added: "+3V3"
- board text added: "FREF_PITCH"
- board text added: "FREF_VOLUME"
- board text added: "F_REF"
- board text added: "GND"
- board text added: "HETERODYNE_OUT"
- board text added: "OSC"
- board text added: "OSC_P"
- board text added: "OSC_V"
- board text added: "PIT"
- board text added: "PITCH SENSOR"
- board text added: "PITCH_HOUT"
- board text added: "PREF"
- board text added: "Teensy Theremin Heterodyne rev 0.1 U1: ADG721BRMZ U2, U3: LVC2G04"
- board text added: "VOL"
- board text added: "VOLUME SENSOR"
- board text added: "VOL_HOUT"
- board text added: "VREF"
