File: teensy4theremin/kicad/sensor/teensy41_display_controls/teensy41_display_controls.kicad_pcb (KiCad board)
At the start: 2 copper layers, 135.9 x 78.7 mm, 14 parts, among them J1 Conn_02x15_Odd_Even, SW1 Rotary_Encoder_Switch, SW2 Rotary_Encoder_Switch, SW3 Rotary_Encoder_Switch, SW4 Rotary_Encoder_Switch, SW5 SW_Push, SW6 SW_Push, SW7 SW_Push, U1 TeensyLCD

Commit message: teensy 41 theremin main board and display board rev 0.1
Parts:
- added C1: 0.1uF, Capacitor_SMD:C_0805_2012Metric_Pad1.18x1.45mm_HandSolder, B.Cu at (67.1, 105.4)
- added C10: 0.01uF, Capacitor_SMD:C_0805_2012Metric_Pad1.18x1.45mm_HandSolder, B.Cu at (61.0, 82.8)
- added C11: 0.01uF, Capacitor_SMD:C_0805_2012Metric_Pad1.18x1.45mm_HandSolder, B.Cu at (64.4, 55.2)
- added C12: 0.01uF, Capacitor_SMD:C_0805_2012Metric_Pad1.18x1.45mm_HandSolder, B.Cu at (61.0, 45.7)
- added C13: 0.01uF, Capacitor_SMD:C_0805_2012Metric_Pad1.18x1.45mm_HandSolder, B.Cu at (81.3, 105.2)
- added C14: 0.01uF, Capacitor_SMD:C_0805_2012Metric_Pad1.18x1.45mm_HandSolder, B.Cu at (96.5, 105.2)
- added C15: 0.01uF, Capacitor_SMD:C_0805_2012Metric_Pad1.18x1.45mm_HandSolder, B.Cu at (100.3, 105.2)
- added C16: 0.01uF, Capacitor_SMD:C_0805_2012Metric_Pad1.18x1.45mm_HandSolder, B.Cu at (115.6, 105.2)
- added C17: 0.01uF, Capacitor_SMD:C_0805_2012Metric_Pad1.18x1.45mm_HandSolder, B.Cu at (119.4, 105.2)
- added C18: 0.01uF, Capacitor_SMD:C_0805_2012Metric_Pad1.18x1.45mm_HandSolder, B.Cu at (134.6, 105.2)
- added C19: 0.01uF, Capacitor_SMD:C_0805_2012Metric_Pad1.18x1.45mm_HandSolder, B.Cu at (91.4, 89.9)
- added C2: 0.1uF, Capacitor_SMD:C_0805_2012Metric_Pad1.18x1.45mm_HandSolder, B.Cu at (165.1, 52.1)
- added C20: 0.01uF, Capacitor_SMD:C_0805_2012Metric_Pad1.18x1.45mm_HandSolder, B.Cu at (110.5, 89.9)
- added C21: 0.01uF, Capacitor_SMD:C_0805_2012Metric_Pad1.18x1.45mm_HandSolder, B.Cu at (129.5, 89.9)
- added C22: 0.01uF, Capacitor_SMD:C_0805_2012Metric_Pad1.18x1.45mm_HandSolder, B.Cu at (138.4, 105.2)
- added C23: 0.01uF, Capacitor_SMD:C_0805_2012Metric_Pad1.18x1.45mm_HandSolder, B.Cu at (153.7, 105.2)
- added C24: 0.01uF, Capacitor_SMD:C_0805_2012Metric_Pad1.18x1.45mm_HandSolder, B.Cu at (148.6, 90.2)
- added C25: 0.1uF, Capacitor_SMD:C_0805_2012Metric_Pad1.18x1.45mm_HandSolder, B.Cu at (77.5, 108.0)
- added C26: 0.1uF, Capacitor_SMD:C_0805_2012Metric_Pad1.18x1.45mm_HandSolder, B.Cu at (159.4, 76.2)
- added C3: 0.1uF, Capacitor_SMD:C_0805_2012Metric_Pad1.18x1.45mm_HandSolder, B.Cu at (165.1, 69.8)
- added C4: 0.1uF, Capacitor_SMD:C_0805_2012Metric_Pad1.18x1.45mm_HandSolder, B.Cu at (165.1, 87.6)
- added C5: 0.1uF, Capacitor_SMD:C_0805_2012Metric_Pad1.18x1.45mm_HandSolder, B.Cu at (165.1, 105.4)
- added C6: 1uF, Capacitor_SMD:C_0805_2012Metric_Pad1.18x1.45mm_HandSolder, B.Cu at (74.9, 83.8)
- added C7: 1uF, Capacitor_SMD:C_0805_2012Metric_Pad1.18x1.45mm_HandSolder, B.Cu at (80.0, 49.5)
- added C8: 0.1uF, Capacitor_SMD:C_0805_2012Metric_Pad1.18x1.45mm_HandSolder, B.Cu at (72.6, 86.4)
- added C9: 0.1uF, Capacitor_SMD:C_0805_2012Metric_Pad1.18x1.45mm_HandSolder, B.Cu at (76.4, 49.5)
- added R1: 100, Resistor_SMD:R_0805_2012Metric_Pad1.20x1.40mm_HandSolder, B.Cu at (80.0, 54.6)
- added R10: 10K, Resistor_SMD:R_0805_2012Metric_Pad1.20x1.40mm_HandSolder, B.Cu at (104.4, 104.1)
- added R11: 10K, Resistor_SMD:R_0805_2012Metric_Pad1.20x1.40mm_HandSolder, B.Cu at (111.5, 104.1)
- added R12: 10K, Resistor_SMD:R_0805_2012Metric_Pad1.20x1.40mm_HandSolder, B.Cu at (123.5, 104.1)
- added R13: 10K, Resistor_SMD:R_0805_2012Metric_Pad1.20x1.40mm_HandSolder, B.Cu at (130.5, 104.1)
- added R14: 10K, Resistor_SMD:R_0805_2012Metric_Pad1.20x1.40mm_HandSolder, B.Cu at (86.4, 98.8)
- added R15: 10K, Resistor_SMD:R_0805_2012Metric_Pad1.20x1.40mm_HandSolder, B.Cu at (91.4, 98.8)
- added R16: 10K, Resistor_SMD:R_0805_2012Metric_Pad1.20x1.40mm_HandSolder, B.Cu at (105.4, 98.8)
- added R17: 10K, Resistor_SMD:R_0805_2012Metric_Pad1.20x1.40mm_HandSolder, B.Cu at (110.5, 98.8)
- added R18: 10K, Resistor_SMD:R_0805_2012Metric_Pad1.20x1.40mm_HandSolder, B.Cu at (124.5, 98.8)
- added R19: 10K, Resistor_SMD:R_0805_2012Metric_Pad1.20x1.40mm_HandSolder, B.Cu at (129.5, 98.8)
- added R2: 10K, Resistor_SMD:R_0805_2012Metric_Pad1.20x1.40mm_HandSolder, B.Cu at (70.1, 83.8)
- added R20: 10K, Resistor_SMD:R_0805_2012Metric_Pad1.20x1.40mm_HandSolder, B.Cu at (86.4, 89.9)
- added R21: 10K, Resistor_SMD:R_0805_2012Metric_Pad1.20x1.40mm_HandSolder, B.Cu at (105.4, 89.9)
- added R22: 10K, Resistor_SMD:R_0805_2012Metric_Pad1.20x1.40mm_HandSolder, B.Cu at (124.5, 89.9)
- added R23: 10K, Resistor_SMD:R_0805_2012Metric_Pad1.20x1.40mm_HandSolder, B.Cu at (88.9, 96.8)
- added R24: 10K, Resistor_SMD:R_0805_2012Metric_Pad1.20x1.40mm_HandSolder, B.Cu at (108.0, 96.8)
- added R25: 10K, Resistor_SMD:R_0805_2012Metric_Pad1.20x1.40mm_HandSolder, B.Cu at (127.0, 96.8)
- added R26: 10K, Resistor_SMD:R_0805_2012Metric_Pad1.20x1.40mm_HandSolder, B.Cu at (142.5, 104.1)
- added R27: 10K, Resistor_SMD:R_0805_2012Metric_Pad1.20x1.40mm_HandSolder, B.Cu at (149.6, 104.1)
- added R28: 10K, Resistor_SMD:R_0805_2012Metric_Pad1.20x1.40mm_HandSolder, B.Cu at (143.5, 98.8)
- added R29: 10K, Resistor_SMD:R_0805_2012Metric_Pad1.20x1.40mm_HandSolder, B.Cu at (148.6, 98.8)
- added R3: 10K, Resistor_SMD:R_0805_2012Metric_Pad1.20x1.40mm_HandSolder, B.Cu at (68.6, 58.1)
- added R30: 10K, Resistor_SMD:R_0805_2012Metric_Pad1.20x1.40mm_HandSolder, B.Cu at (143.5, 90.2)
- added R31: 10K, Resistor_SMD:R_0805_2012Metric_Pad1.20x1.40mm_HandSolder, B.Cu at (146.1, 96.8)
- added R4: 10K, Resistor_SMD:R_0805_2012Metric_Pad1.20x1.40mm_HandSolder, B.Cu at (68.6, 54.2)
- added R5: 10K, Resistor_SMD:R_0805_2012Metric_Pad1.20x1.40mm_HandSolder, B.Cu at (66.0, 82.8)
- added R6: 10K, Resistor_SMD:R_0805_2012Metric_Pad1.20x1.40mm_HandSolder, B.Cu at (64.4, 59.1)
- added R7: 10K, Resistor_SMD:R_0805_2012Metric_Pad1.20x1.40mm_HandSolder, B.Cu at (65.0, 47.0)
- added R8: 10K, Resistor_SMD:R_0805_2012Metric_Pad1.20x1.40mm_HandSolder, B.Cu at (85.4, 104.1)
- added R9: 10K, Resistor_SMD:R_0805_2012Metric_Pad1.20x1.40mm_HandSolder, B.Cu at (92.4, 104.1)
- J1: value Conn_02x15_Odd_Even -> MCU_CONN
- RV1, RV2, RV3, RV4, RV5: value R_POT -> 25K
- SW1: value Rotary_Encoder_Switch -> ENC1
- SW2: value Rotary_Encoder_Switch -> ENC2
- SW3: value Rotary_Encoder_Switch -> ENC3
- SW4: value Rotary_Encoder_Switch -> ENC4
- SW5: value SW_Push -> BTN1
- SW6: value SW_Push -> BTN2
- SW7: value SW_Push -> BTN3
- moved RV5 97.8 mm to (168.9, 108.0)
- moved RV1 97.8 mm to (71.1, 108.0)
Connections:
- J1 pad 1: Net-(J1-Pad1) -> +5V
- J1 pad 10: Net-(J1-Pad10) -> /T_IRQ
- J1 pad 11: Net-(J1-Pad11) -> /LCD_CS
- J1 pad 12: Net-(J1-Pad12) -> /MOSI
- J1 pad 13: Net-(J1-Pad13) -> /SCK
- J1 pad 14: Net-(J1-Pad14) -> /MISO
- J1 pad 15: Net-(J1-Pad15) -> +3V3
- J1 pad 16: Net-(J1-Pad16) -> /POT1
- J1 pad 17: Net-(J1-Pad17) -> /ENC1_C
- J1 pad 18: Net-(J1-Pad18) -> /POT2
- J1 pad 19: Net-(J1-Pad19) -> /ENC2_C
- J1 pad 2: Net-(J1-Pad2) -> GND
- J1 pad 20: Net-(J1-Pad20) -> /POT3
- J1 pad 21: Net-(J1-Pad21) -> /ENC3_C
- J1 pad 22: Net-(J1-Pad22) -> /POT4
- J1 pad 23: Net-(J1-Pad23) -> /ENC4_C
- J1 pad 24: Net-(J1-Pad24) -> /POT5
- J1 pad 25: Net-(J1-Pad25) -> /ENC4_A
- J1 pad 26: Net-(J1-Pad26) -> /T_CS
- J1 pad 27: Net-(J1-Pad27) -> /ENC4_B
- J1 pad 28: Net-(J1-Pad28) -> /BTN1
- J1 pad 29: Net-(J1-Pad29) -> /BTN3
- J1 pad 3: Net-(J1-Pad3) -> /ENC1_A
- J1 pad 30: Net-(J1-Pad30) -> /BTN2
- J1 pad 4: Net-(J1-Pad4) -> /ENC1_B
- J1 pad 5: Net-(J1-Pad5) -> /ENC2_A
- J1 pad 6: Net-(J1-Pad6) -> /ENC2_B
- J1 pad 7: Net-(J1-Pad7) -> /ENC3_A
- J1 pad 8: Net-(J1-Pad8) -> /ENC3_B
- J1 pad 9: Net-(J1-Pad9) -> /LCD_DC
- RV1 pad 1: Net-(RV1-Pad1) -> +3V3
- RV1 pad 2: Net-(RV1-Pad2) -> /POT1
- RV1 pad 3: Net-(RV1-Pad3) -> GND
- RV2 pad 1: Net-(RV2-Pad1) -> +3V3
- RV2 pad 2: Net-(RV2-Pad2) -> /POT2
- RV2 pad 3: Net-(RV2-Pad3) -> GND
- RV3 pad 1: Net-(RV3-Pad1) -> +3V3
- RV3 pad 2: Net-(RV3-Pad2) -> /POT3
- RV3 pad 3: Net-(RV3-Pad3) -> GND
- RV4 pad 1: Net-(RV4-Pad1) -> +3V3
- RV4 pad 2: Net-(RV4-Pad2) -> /POT4
- RV4 pad 3: Net-(RV4-Pad3) -> GND
- RV5 pad 1: Net-(RV5-Pad1) -> +3V3
- RV5 pad 2: Net-(RV5-Pad2) -> /POT5
- RV5 pad 3: Net-(RV5-Pad3) -> GND
- SW1 pad C: Net-(SW1-PadC) -> GND
- SW1 pad S1: Net-(SW1-PadS1) -> GND
- SW2 pad C: Net-(SW2-PadC) -> GND
- SW2 pad S1: Net-(SW2-PadS1) -> GND
- SW3 pad C: Net-(SW3-PadC) -> GND
- SW3 pad S1: Net-(SW3-PadS1) -> GND
- SW4 pad C: Net-(SW4-PadC) -> GND
- SW4 pad S1: Net-(SW4-PadS1) -> GND
- SW5 pad 1: Net-(SW5-Pad1) -> GND
- SW6 pad 1: Net-(SW6-Pad1) -> GND
- SW7 pad 1: Net-(SW7-Pad1) -> GND
- U1 pad 1: Net-(U1-Pad1) -> +5V
- U1 pad 10: Net-(U1-Pad10) -> /SCK
- U1 pad 11: Net-(U1-Pad11) -> /T_CS
- U1 pad 12: Net-(U1-Pad12) -> /MOSI
- U1 pad 13: Net-(U1-Pad13) -> /MISO
- U1 pad 14: Net-(U1-Pad14) -> /T_IRQ
- U1 pad 2: Net-(U1-Pad2) -> GND
- U1 pad 3: Net-(U1-Pad3) -> /LCD_CS
- U1 pad 4: Net-(U1-Pad4) -> +3V3
- U1 pad 5: Net-(U1-Pad5) -> /LCD_DC
- U1 pad 6: Net-(U1-Pad6) -> /MOSI
- U1 pad 7: Net-(U1-Pad7) -> /SCK
- U1 pad 9: Net-(U1-Pad9) -> /MISO
Routing:
- net GND: track 0.00 -> 584.6 mm, vias 0 -> 8
- net +3V3: track 0.00 -> 469.3 mm, vias 0 -> 10
- net /POT3: track 0.00 -> 185.0 mm
- net /POT2: track 0.00 -> 159.0 mm
- net /POT4: track 0.00 -> 149.1 mm, vias 0 -> 1
- net /POT5: track 0.00 -> 134.2 mm
- net /ENC3_B: track 0.00 -> 118.3 mm, vias 0 -> 2
- net /ENC1_B: track 0.00 -> 106.1 mm, vias 0 -> 1
- net /ENC4_B: track 0.00 -> 104.5 mm, vias 0 -> 1
- net /ENC2_B: track 0.00 -> 102.8 mm, vias 0 -> 2
- net /ENC4_C: track 0.00 -> 102.1 mm, vias 0 -> 1
- net /ENC3_A: track 0.00 -> 98.7 mm, vias 0 -> 2
- net /ENC4_A: track 0.00 -> 97.2 mm, vias 0 -> 1
- net /ENC1_A: track 0.00 -> 83.8 mm, vias 0 -> 1
- net /ENC2_A: track 0.00 -> 82.2 mm, vias 0 -> 2
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- added copper zone on B.Cu, net GND
- added copper zone on F.Cu, net GND
Other:
- outline, holes or cut-outs redrawn
- board text added: "+3.3V"
- board text added: "+5V"
- board text added: "BTN1"
- board text added: "BTN2"
- board text added: "BTN3"
- board text added: "Color Touch LCD pjrc.com"
- board text added: "ENC1A"
- board text added: "ENC1B"
- board text added: "ENC1C"
- board text added: "ENC2A"
- board text added: "ENC2B"
- board text added: "ENC2C"
- board text added: "ENC3A"
- board text added: "ENC3B"
- board text added: "ENC3C"
- board text added: "ENC4A"
- board text added: "ENC4B"
- board text added: "ENC4C"
- board text added: "GND"
- board text added: "LCD_CS"
- board text added: "LCD_DC"
- board text added: "MISO"
- board text added: "MOSI"
- board text added: "POT1"
- board text added: "POT2"
- board text added: "POT3"
- board text added: "POT4"
- board text added: "POT5"
- board text added: "SCK"
- board text added: "T_CS"
- board text added: "T_IRQ"
- board text added: "Teensy 4 Theremin Display and Controls Board"

Commit message: update PCBs
Parts:
- RV1, RV2, RV3, RV4, RV5: footprint Potentiometer_THT:Potentiometer_Bourns_PTV09A-1_Single_Vertical -> Potentiometer_THT:Potentiometer_TT_P0915N
- moved C6 7.77 mm to (73.4, 91.4), turned to 180 degrees
- moved RV4 5.04 mm to (163.8, 90.2), turned to 0 degrees
- moved RV5 5.04 mm to (163.9, 108.0), turned to 0 degrees
- moved RV1 5.00 mm to (66.1, 108.0), turned to 0 degrees
- moved RV2 5.00 mm to (163.9, 54.6), turned to 0 degrees
- moved RV3 5.00 mm to (163.9, 72.4), turned to 0 degrees
- moved C8 1.56 mm to (71.1, 86.8), turned to 270 degrees
Connections:
- RV1 pad 1: +3V3 -> GND
- RV1 pad 3: GND -> +3V3
- RV2 pad 1: +3V3 -> GND
- RV2 pad 3: GND -> +3V3
- RV3 pad 1: +3V3 -> GND
- RV3 pad 3: GND -> +3V3
- RV4 pad 1: +3V3 -> GND
- RV4 pad 3: GND -> +3V3
- RV5 pad 1: +3V3 -> GND
- RV5 pad 3: GND -> +3V3
Routing:
- net GND: track 584.6 -> 572.0 mm, vias 8 -> 9
- net +3V3: track 469.3 -> 470.8 mm, vias 10 -> 11
- net Net-(R2-Pad1): track 9.47 -> 10.7 mm
Other:
- board text added: "Teensy 4 Theremin Display and Controls Board rev 1.2"
- board text removed: "Teensy 4 Theremin Display and Controls Board"
