File: teensy4theremin/kicad/mainboard/teensy41_main_board_v2/teensy41_main_board_v2.kicad_pcb (KiCad board)
At the start: 2 copper layers, 121.9 x 61 mm, 77 parts, among them J1 LCD_CONTROLS, J10 LINEOUT, J11 Grounding, J12 PHONES, J13 LINEIN, J14 Grounding2, J2 LINE_IN, J3 LINE_OUT_BIG, J4 VOL_SENSOR, J5 PITCH_SENSOR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

Commit message: update sensor schematics and model:
Parts:
- added R18: 2.2K, Resistor_SMD:R_0805_2012Metric_Pad1.20x1.40mm_HandSolder, B.Cu at (102.4, 108.7)
- added R19: 2.2K, Resistor_SMD:R_0805_2012Metric_Pad1.20x1.40mm_HandSolder, B.Cu at (104.4, 108.7)
- added R20: 100 *, Resistor_SMD:R_0805_2012Metric_Pad1.20x1.40mm_HandSolder, B.Cu at (45.7, 116.6)
- added R21: 100 *, Resistor_SMD:R_0805_2012Metric_Pad1.20x1.40mm_HandSolder, B.Cu at (90.8, 120.9)
- C10, C11: value 1uF -> 10uF; footprint Capacitor_SMD:C_0805_2012Metric_Pad1.18x1.45mm_HandSolder -> Capacitor_Tantalum_SMD:CP_EIA-3216-18_Kemet-A_Pad1.58x1.35mm_HandSolder
- R2, R3, R4, R5: value 110 -> 100 *
- moved C2 2.54 mm to (99.1, 116.8)
- moved C4 2.54 mm to (99.1, 125.1)
- moved C6 2.54 mm to (99.1, 119.4)
- moved J5 2.54 mm to (94.0, 118.1)
- moved U5 2.54 mm to (99.1, 122.2)
- moved J11 1.91 mm to (42.5, 78.7)
- moved J14 1.91 mm to (42.5, 83.8)
- moved C10 0.48 mm to (51.9, 120.1)
- moved C11 0.15 mm to (81.4, 125.7)
Routing:
- net GND: track 586.1 -> 631.4 mm, vias 21 -> 30
- net /VCC_VOL: track 26.0 -> 37.3 mm, vias 1 -> 4
- net /I2C_SDA: track 41.6 -> 49.5 mm
- net /3V3: track 303.6 -> 310.4 mm, vias 11 -> 13
- net /I2C_SCL: track 50.1 -> 56.2 mm
- net /VCC_PITCH: track 17.2 -> 20.3 mm
- net /N_VOL: track 11.8 -> 14.7 mm
- net /N_PITCH: track 6.66 -> 9.34 mm
- net /P_PITCH: track 12.1 -> 14.7 mm
- net /VIN: track 183.8 -> 182.6 mm
- net /P_VOL: track 22.2 -> 23.4 mm
- net /AVCC: vias 6 -> 7
- added copper zone on F.Cu, net /3V3
- added copper zone on B.Cu, net /VCC_VOL
Other:
- board text added: "+"
- board text added: "+4.7"
- board text added: "G"
- board text added: "L"
- board text added: "PITCH SENSOR"
- board text added: "R"
- board text added: "VOLUME SENSOR"
- board text added: "WM8731"
