File: teensy4theremin/kicad/mainboard/teensy41_main_board_v2/teensy41_main_board_v2.sch (KiCad schematic (older format))
At the start: 77 parts, among them J1 LCD_CONTROLS, J10 LINEOUT, J11 Grounding, J12 PHONES, J13 LINEIN, J14 Grounding2, J2 LINE_IN, J3 LINE_OUT_BIG, J4 VOL_SENSOR, J5 PITCH_SENSOR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

Commit message: update sensor schematics and model:
Parts:
- removed C10, C11: 1uF, Capacitor_SMD:C_0805_2012Metric_Pad1.18x1.45mm_HandSolder, symbol Device:C
- added C10, C11: 10uF, Capacitor_Tantalum_SMD:CP_EIA-3216-18_Kemet-A_Pad1.58x1.35mm_HandSolder, symbol Device:CP
- added R18, R19: 2.2K, Resistor_SMD:R_0805_2012Metric_Pad1.20x1.40mm_HandSolder, symbol Device:R
- added R20, R21: 100 *, Resistor_SMD:R_0805_2012Metric_Pad1.20x1.40mm_HandSolder, symbol Device:R
- R2, R3, R4, R5: value 110 -> 100 *
Connections:
- net 3V3: now also C10.1, C11.1, R18.1, R19.1
- net GND: now also C10.2, C11.2
- net I2C_SCL: now also R18.2
- net I2C_SDA: now also R19.2
- net N_PITCH: now also R21.2
- net N_VOL: now also R20.2
- net P_PITCH: now also R21.1
- net P_VOL: now also R20.1
Other:
- moved on the sheet: R2, R3, R4, R5
