File: teensy4theremin/kicad/sensor/current_sensing_bjt/current_sensing_bjt.kicad_pcb (KiCad board)
At the start: 2 copper layers, 70.5 x 21.1 mm, 24 parts, among them J1 ANTENNA, J3 INDUCTOR_IN, J6 OSC, Q1 BC549, Q2 BC549, Q3 BC549, Q4 BC549, Q5 BC549, Q6 BC549, Q7 BC549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

Commit message: update sensor schematics and model:
Parts:
- added Q9: BC549, Package_TO_SOT_THT:TO-92_Inline_Wide, F.Cu at (137.2, 106.7)
- R5: value 680 -> 100; footprint Resistor_THT:R_Axial_DIN0207_L6.3mm_D2.5mm_P10.16mm_Horizontal -> Resistor_THT:R_Axial_DIN0204_L3.6mm_D1.6mm_P2.54mm_Vertical
Connections:
- Q8 pad 3: /OUT -> Net-(Q8-Pad3)
- R5 pad 2: GND -> Net-(Q8-Pad3)
Routing:
- net /OUT: track 16.3 -> 8.67 mm
- net Net-(Q8-Pad3): track 0.00 -> 7.62 mm
- net Net-(Q5-Pad1): track 12.7 -> 17.8 mm
Changed lines of the file:
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@@
     (thickness 1.6)
     (drawings 21)
-    (tracks 75)
+    (tracks 77)
     (zones 0)
-    (modules 24)
-    (nets 13)
+    (modules 25)
+    (nets 14)
   )
   (page A4)
@@
   )
   (setup
-    (last_trace_width 0.5)
+    (last_trace_width 0.25)
     (user_trace_width 0.5)
     (trace_clearance 0.2)
@@
   (net 11 "Net-(Q5-Pad1)")
   (net 12 "Net-(C2-Pad1)")
+  (net 13 "Net-(Q8-Pad3)")
   (net_class Default "This is the default net class."
     (clearance 0.2)
@@
     (add_net "Net-(Q4-Pad2)")
     (add_net "Net-(Q5-Pad1)")
+    (add_net "Net-(Q8-Pad3)")
     (add_net VCC)
+  )
+  (module Resistor_THT:R_Axial_DIN0204_L3.6mm_D1.6mm_P2.54mm_Vertical (layer F.Cu)
+    (at 137.16 101.6 270)
+    (descr "Resistor, Axial_DIN0204 series, Axial, Vertical, pin pitch=2.54mm, 0.167W, length*diameter=3.6*1.6mm^2, http://cdn-reichelt.de/documents/datenblatt/B400/1_4W%23YAG.pdf")
+    (tags "Resistor Axial_DIN0204 series Axial Vertical pin pitch 2.54mm 0.167W length 3.6mm diameter 1.6mm")
+    (fp_text reference R5 (at 1.27 -1.92 90) (layer F.SilkS)
+      (effects (font (size 1 1) (thickness 0.15)))
+    )
+    (fp_text value 100 (at 1.27 1.92 90) (layer F.Fab)
+      (effects (font (size 1 1) (thickness 0.15)))
+    )
+    (fp_text user %R (at 1.27 -1.92 90) (layer F.Fab)
+      (effects (font (size 1 1) (thickness 0.15)))
+    )
+    (fp_circle (center 0 0) (end 0.8 0) (layer F.Fab) (width 0.1))
+    (fp_circle (center 0 0) (end 0.92 0) (layer F.SilkS) (width 0.12))
+    (fp_line (start 0 0) (end 2.54 0) (layer F.Fab) (width 0.1))
+    (fp_line (start 0.92 0) (end 1.54 0) (layer F.SilkS) (width 0.12))
+    (fp_line (start -1.05 -1.05) (end -1.05 1.05) (layer F.CrtYd) (width 0.05))
+    (fp_line (start -1.05 1.05) (end 3.49 1.05) (layer F.CrtYd) (width 0.05))
+    (fp_line (start 3.49 1.05) (end 3.49 -1.05) (layer F.CrtYd) (width 0.05))
+    (fp_line (start 3.49 -1.05) (end -1.05 -1.05) (layer F.CrtYd) (width 0.05))
+    (pad 2 thru_hole oval (at 2.54 0 270) (size 1.4 1.4) (drill 0.7) (layers *.Cu *.Mask)
+      (net 13 "Net-(Q8-Pad3)"))
+    (pad 1 thru_hole circle (at 0 0 270) (size 1.4 1.4) (drill 0.7) (layers *.Cu *.Mask)
+      (net 6 /OUT))
+    (model ${KISYS3DMOD}/Resistor_THT.3dshapes/R_Axial_DIN0204_L3.6mm_D1.6mm_P2.54mm_Vertical.wrl
+      (at (xyz 0 0 0))
+      (scale (xyz 1 1 1))
+      (rotate (xyz 0 0 0))
+    )
+  )
+  (module Package_TO_SOT_THT:TO-92_Inline_Wide (layer F.Cu)
+    (at 137.16 106.68 270)
+    (descr "TO-92 leads in-line, wide, drill 0.75mm (see NXP sot054_po.pdf)")
+    (tags "to-92 sc-43 sc-43a sot54 PA33 transistor")
+    (fp_text reference Q9 (at 2.54 -3.56 90) (layer F.SilkS)
+      (effects (font (size 1 1) (thickness 0.15)))
+    )
+    (fp_text value BC549 (at 2.54 2.79 90) (layer F.Fab)
+      (effects (font (size 1 1) (thickness 0.15)))
+    )
+    (fp_arc (start 2.54 0) (end 4.34 1.85) (angle -20) (layer F.SilkS) (width 0.12))
+    (fp_arc (start 2.54 0) (end 2.54 -2.48) (angle -135) (layer F.Fab) (width 0.1))
+    (fp_arc (start 2.54 0) (end 2.54 -2.48) (angle 135) (layer F.Fab) (width 0.1))
+    (fp_arc (start 2.54 0) (end 2.54 -2.6) (angle 65) (layer F.SilkS) (width 0.12))
+    (fp_arc (start 2.54 0) (end 2.54 -2.6) (angle -65) (layer F.SilkS) (width 0.12))
+    (fp_arc (start 2.54 0) (end 0.74 1.85) (angle 20) (layer F.SilkS) (width 0.12))
+    (fp_text user %R (at 2.54 0 90) (layer F.Fab)
+      (effects (font (size 1 1) (thickness 0.15)))
+    )
+    (fp_line (start 0.74 1.85) (end 4.34 1.85) (layer F.SilkS) (width 0.12))
+    (fp_line (start 0.8 1.75) (end 4.3 1.75) (layer F.Fab) (width 0.1))
+    (fp_line (start -1.01 -2.73) (end 6.09 -2.73) (layer F.CrtYd) (width 0.05))
+    (fp_line (start -1.01 -2.73) (end -1.01 2.01) (layer F.CrtYd) (width 0.05))
+    (fp_line (start 6.09 2.01) (end 6.09 -2.73) (layer F.CrtYd) (width 0.05))
+    (fp_line (start 6.09 2.01) (end -1.01 2.01) (layer F.CrtYd) (width 0.05))
+    (pad 1 thru_hole rect (at 0 0 270) (size 1.5 1.5) (drill 0.8) (layers *.Cu *.Mask)
+      (net 13 "Net-(Q8-Pad3)"))
+    (pad 3 thru_hole circle (at 5.08 0 270) (size 1.5 1.5) (drill 0.8) (layers *.Cu *.Mask)
+      (net 1 GND))
+    (pad 2 thru_hole circle (at 2.54 0 270) (size 1.5 1.5) (drill 0.8) (layers *.Cu *.Mask)
+      (net 11 "Net-(Q5-Pad1)"))
+    (model ${KISYS3DMOD}/Package_TO_SOT_THT.3dshapes/TO-92_Inline_Wide.wrl
+      (at (xyz 0 0 0))
+      (scale (xyz 1 1 1))
+      (rotate (xyz 0 0 0))
+    )
   )
   (module Connector_PinHeader_2.54mm:PinHeader_1x01_P2.54mm_Vertical (layer F.Cu)
@@
       (net 4 VCC))
     (pad 3 thru_hole circle (at 5.08 0 270) (size 1.5 1.5) (drill 0.8) (layers *.Cu *.Mask)
-      (net 6 /OUT))
+      (net 13 "Net-(Q8-Pad3)"))
     (pad 2 thru_hole circle (at 2.54 0 270) (size 1.5 1.5) (drill 0.8) (layers *.Cu *.Mask)
       (net 10 "Net-(Q4-Pad2)"))
@@
   )
   (module Resistor_THT:R_Axial_DIN0207_L6.3mm_D2.5mm_P10.16mm_Horizontal (layer F.Cu)
-    (at 137.16 101.6 270)
-    (descr "Resistor, Axial_DIN0207 series, Axial, Horizontal, pin pitch=10.16mm, 0.25W = 1/4W, length*diameter=6.3*2.5mm^2, http://cdn-reichelt.de/documents/datenblatt/B400/1_4W%23YAG.pdf")
-    (tags "Resistor Axial_DIN0207 series Axial Horizontal pin pitch 10.16mm 0.25W = 1/4W length 6.3mm diameter 2.5mm")
-    (fp_text reference R5 (at 5.08 0 90) (layer F.SilkS)
-      (effects (font (size 1 1) (thickness 0.15)))
-    )
-    (fp_text value 680 (at 5.08 2.37 90) (layer F.Fab)
-      (effects (font (size 1 1) (thickness 0.15)))
-    )
-    (fp_text user %R (at 5.08 0 90) (layer F.Fab)
-      (effects (font (size 1 1) (thickness 0.15)))
-    )
-    (fp_line (start 1.93 -1.25) (end 1.93 1.25) (layer F.Fab) (width 0.1))
-    (fp_line (start 1.93 1.25) (end 8.23 1.25) (layer F.Fab) (width 0.1))
-    (fp_line (start 8.23 1.25) (end 8.23 -1.25) (layer F.Fab) (width 0.1))
-    (fp_line (start 8.23 -1.25) (end 1.93 -1.25) (layer F.Fab) (width 0.1))
-    (fp_line (start 0 0) (end 1.93 0) (layer F.Fab) (width 0.1))
-    (fp_line (start 10.16 0) (end 8.23 0) (layer F.Fab) (width 0.1))
-    (fp_line (start 1.81 -1.37) (end 1.81 1.37) (layer F.SilkS) (width 0.12))
-    (fp_line (start 1.81 1.37) (end 8.35 1.37) (layer F.SilkS) (width 0.12))
-    (fp_line (start 8.35 1.37) (end 8.35 -1.37) (layer F.SilkS) (width 0.12))
-    (fp_line (start 8.35 -1.37) (end 1.81 -1.37) (layer F.SilkS) (width 0.12))
-    (fp_line (start 1.04 0) (end 1.81 0) (layer F.SilkS) (width 0.12))
-    (fp_line (start 9.12 0) (end 8.35 0) (layer F.SilkS) (width 0.12))
-    (fp_line (start -1.05 -1.5) (end -1.05 1.5) (layer F.CrtYd) (width 0.05))
-    (fp_line (start -1.05 1.5) (end 11.21 1.5) (layer F.CrtYd) (width 0.05))
-    (fp_line (start 11.21 1.5) (end 11.21 -1.5) (layer F.CrtYd) (width 0.05))
-    (fp_line (start 11.21 -1.5) (end -1.05 -1.5) (layer F.CrtYd) (width 0.05))
-    (pad 2 thru_hole oval (at 10.16 0 270) (size 1.6 1.6) (drill 0.8) (layers *.Cu *.Mask)
-      (net 1 GND))
-    (pad 1 thru_hole circle (at 0 0 270) (size 1.6 1.6) (drill 0.8) (layers *.Cu *.Mask)
-      (net 6 /OUT))
-    (model ${KISYS3DMOD}/Resistor_THT.3dshapes/R_Axial_DIN0207_L6.3mm_D2.5mm_P10.16mm_Horizontal.wrl
-      (at (xyz 0 0 0))
-      (scale (xyz 1 1 1))
-      (rotate (xyz 0 0 0))
-    )
-  )
-  (module Resistor_THT:R_Axial_DIN0207_L6.3mm_D2.5mm_P10.16mm_Horizontal (layer F.Cu)
     (at 121.92 99.06 270)
     (descr "Resistor, Axial_DIN0207 series, Axial, Horizontal, pin pitch=10.16mm, 0.25W = 1/4W, length*diameter=6.3*2.5mm^2, http://cdn-reichelt.de/documents/datenblatt/B400/1_4W%23YAG.pdf")
@@
   (segment (start 107.95 99.06) (end 106.68 97.79) (width 0.25) (layer F.Cu) (net 5))
   (segment (start 109.22 99.06) (end 107.95 99.06) (width 0.25) (layer F.Cu) (net 5))
-  (segment (start 132.08 104.14) (end 137.16 104.14) (width 0.5) (layer B.Cu) (net 6))
-  (segment (start 137.16 104.14) (end 137.16 101.6) (width 0.5) (layer B.Cu) (net 6))
-  (segment (start 144.78 104.14) (end 139.7 104.14) (width 0.25) (layer F.Cu) (net 6))
-  (segment (start 139.7 104.14) (end 137.16 101.6) (width 0.25) (layer F.Cu) (net 6))
+  (segment (start 137.16 101.6) (end 139.7 101.6) (width 0.25) (layer F.Cu) (net 6))
+  (segment (start 139.7 101.6) (end 142.24 104.14) (width 0.25) (layer F.Cu) (net 6))
+  (segment (start 142.24 104.14) (end 144.78 104.14) (width 0.25) (layer F.Cu) (net 6))
   (segment (start 109.22 109.22) (end 114.3 109.22) (width 0.5) (layer B.Cu) (net 7))
   (segment (start 114.3 109.22) (end 119.38 109.22) (width 0.5) (layer B.Cu) (net 7))
@@
   (segment (start 132.08 109.22) (end 132.08 106.68) (width 0.5) (layer B.Cu) (net 11))
   (segment (start 121.92 109.22) (end 127 109.22) (width 0.5) (layer B.Cu) (net 11))
+  (segment (start 137.16 109.22) (end 132.08 109.22) (width 0.5) (layer B.Cu) (net 11))
   (segment (start 96.52 111.76) (end 99.1 111.76) (width 0.5) (layer B.Cu) (net 12))
   (segment (start 96.52 109.18) (end 96.52 111.76) (width 0.5) (layer B.Cu) (net 12))
+  (segment (start 137.16 106.68) (end 137.16 104.14) (width 0.5) (layer B.Cu) (net 13))
+  (segment (start 132.08 104.14) (end 137.16 104.14) (width 0.5) (layer B.Cu) (net 13))
 )

Commit message: controls board pcb
Other:
- board size 70.5 x 21.1 mm -> 70.5 x 20.4 mm
Changed lines of the file:
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@@
   )
   (gr_circle (center 149.225 111.236) (end 150.325 111.236) (layer Edge.Cuts) (width 0.15))
-  (gr_circle (center 149.225 95.25) (end 150.325 95.25) (layer Edge.Cuts) (width 0.15))
+  (gr_circle (center 149.225 95.885) (end 150.325 95.885) (layer Edge.Cuts) (width 0.15))
   (gr_line (start 81.28 113.776) (end 151.765 113.776) (layer Edge.Cuts) (width 0.2))
-  (gr_circle (center 83.82 95.25) (end 84.92 95.25) (layer Edge.Cuts) (width 0.15))
+  (gr_circle (center 83.82 95.885) (end 84.92 95.885) (layer Edge.Cuts) (width 0.15))
   (gr_circle (center 83.82 111.236) (end 84.92 111.236) (layer Edge.Cuts) (width 0.15))
-  (gr_line (start 81.28 92.71) (end 81.28 113.776) (layer Edge.Cuts) (width 0.2))
-  (gr_line (start 151.765 92.71) (end 151.765 113.776) (layer Edge.Cuts) (width 0.2))
-  (gr_line (start 81.28 92.71) (end 151.765 92.71) (layer Edge.Cuts) (width 0.2))
+  (gr_line (start 81.28 93.345) (end 81.28 113.776) (layer Edge.Cuts) (width 0.2))
+  (gr_line (start 151.765 93.345) (end 151.765 113.776) (layer Edge.Cuts) (width 0.2))
+  (gr_line (start 81.28 93.345) (end 151.765 93.345) (layer Edge.Cuts) (width 0.2))
   (dimension 70.485 (width 0.3) (layer Dwgs.User)
     (gr_text "70.485 mm" (at 116.5225 81.72) (layer Dwgs.User)
@@
     (arrow2b (pts (xy 81.28 83.82) (xy 82.406504 83.233579)))
   )
-  (dimension 20.955 (width 0.3) (layer Dwgs.User)
-    (gr_text "20.955 mm" (at 161.485 103.3145 270) (layer Dwgs.User)
+  (dimension 20.32 (width 0.3) (layer Dwgs.User)
+    (gr_text "20.320 mm" (at 161.485 103.505 270) (layer Dwgs.User)
       (effects (font (size 1.5 1.5) (thickness 0.3)))
     )
-    (feature1 (pts (xy 155.575 113.792) (xy 159.971421 113.792)))
-    (feature2 (pts (xy 155.575 92.837) (xy 159.971421 92.837)))
-    (crossbar (pts (xy 159.385 92.837) (xy 159.385 113.792)))
-    (arrow1a (pts (xy 159.385 113.792) (xy 158.798579 112.665496)))
-    (arrow1b (pts (xy 159.385 113.792) (xy 159.971421 112.665496)))
-    (arrow2a (pts (xy 159.385 92.837) (xy 158.798579 93.963504)))
-    (arrow2b (pts (xy 159.385 92.837) (xy 159.971421 93.963504)))
+    (feature1 (pts (xy 155.575 113.665) (xy 159.971421 113.665)))
+    (feature2 (pts (xy 155.575 93.345) (xy 159.971421 93.345)))
+    (crossbar (pts (xy 159.385 93.345) (xy 159.385 113.665)))
+    (arrow1a (pts (xy 159.385 113.665) (xy 158.798579 112.538496)))
+    (arrow1b (pts (xy 159.385 113.665) (xy 159.971421 112.538496)))
+    (arrow2a (pts (xy 159.385 93.345) (xy 158.798579 94.471504)))
+    (arrow2b (pts (xy 159.385 93.345) (xy 159.971421 94.471504)))
   )
   (segment (start 109.22 111.76) (end 114.3 111.76) (width 0.5) (layer B.Cu) (net 1))
