File: coratheremin/kicad/theremin_sensor_pll_pmod/theremin_sensor_pll_pmod.kicad_pcb (KiCad board)
At the start: 2 copper layers, 33 x 20.3 mm, 18 parts, among them J1 PMOD_A, J2 INDUCTOR, U1 LT1711xMS8, U2 LT1711xMS8, U3 LT1711xMS8

Commit message: controls board pcb
Routing:
- net +3V3: track 73.3 -> 74.9 mm, vias 2 -> 3
- added copper zone on B.Cu, net +3V3
- added copper zone on F.Cu, net +3V3
- added copper zone on F.Cu, net GND
Other:
- board text added: "PMOD"
- board text added: "Theremin Sensor rev 0.1"

Commit message: pcbs updated, jlcpcb prod rev 0.1, gerber files
Other:
- board text added: "D3.4mm"
Changed lines of the file:
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@@
   (general
     (thickness 1.6)
-    (drawings 16)
+    (drawings 22)
     (tracks 188)
     (zones 0)
@@
     )
   )
+  (gr_text D3.4mm (at 73.025 71.12) (layer Dwgs.User)
+    (effects (font (size 1 1) (thickness 0.15)))
+  )
+  (dimension 30.48 (width 0.15) (layer Dwgs.User)
+    (gr_text "30.480 mm" (at 58.42 45.69) (layer Dwgs.User)
+      (effects (font (size 1 1) (thickness 0.15)))
+    )
+    (feature1 (pts (xy 43.18 48.26) (xy 43.18 46.403579)))
+    (feature2 (pts (xy 73.66 48.26) (xy 73.66 46.403579)))
+    (crossbar (pts (xy 73.66 46.99) (xy 43.18 46.99)))
+    (arrow1a (pts (xy 43.18 46.99) (xy 44.306504 46.403579)))
+    (arrow1b (pts (xy 43.18 46.99) (xy 44.306504 47.576421)))
+    (arrow2a (pts (xy 73.66 46.99) (xy 72.533496 46.403579)))
+    (arrow2b (pts (xy 73.66 46.99) (xy 72.533496 47.576421)))
+  )
+  (dimension 2.54 (width 0.15) (layer Dwgs.User)
+    (gr_text "2.540 mm" (at 81.437 68.58 270) (layer Dwgs.User)
+      (effects (font (size 1 1) (thickness 0.15)))
+    )
+    (feature1 (pts (xy 78.74 69.85) (xy 80.723421 69.85)))
+    (feature2 (pts (xy 78.74 67.31) (xy 80.723421 67.31)))
+    (crossbar (pts (xy 80.137 67.31) (xy 80.137 69.85)))
+    (arrow1a (pts (xy 80.137 69.85) (xy 79.550579 68.723496)))
+    (arrow1b (pts (xy 80.137 69.85) (xy 80.723421 68.723496)))
+    (arrow2a (pts (xy 80.137 67.31) (xy 79.550579 68.436504)))
+    (arrow2b (pts (xy 80.137 67.31) (xy 80.723421 68.436504)))
+  )
+  (dimension 15.24 (width 0.15) (layer Dwgs.User)
+    (gr_text "15.240 mm" (at 81.437 59.69 270) (layer Dwgs.User)
+      (effects (font (size 1 1) (thickness 0.15)))
+    )
+    (feature1 (pts (xy 78.74 67.31) (xy 80.723421 67.31)))
+    (feature2 (pts (xy 78.74 52.07) (xy 80.723421 52.07)))
+    (crossbar (pts (xy 80.137 52.07) (xy 80.137 67.31)))
+    (arrow1a (pts (xy 80.137 67.31) (xy 79.550579 66.183496)))
+    (arrow1b (pts (xy 80.137 67.31) (xy 80.723421 66.183496)))
+    (arrow2a (pts (xy 80.137 52.07) (xy 79.550579 53.196504)))
+    (arrow2b (pts (xy 80.137 52.07) (xy 80.723421 53.196504)))
+  )
+  (dimension 2.54 (width 0.15) (layer Dwgs.User)
+    (gr_text "2.540 mm" (at 81.31 50.8 270) (layer Dwgs.User)
+      (effects (font (size 1 1) (thickness 0.15)))
+    )
+    (feature1 (pts (xy 78.74 52.07) (xy 80.596421 52.07)))
+    (feature2 (pts (xy 78.74 49.53) (xy 80.596421 49.53)))
+    (crossbar (pts (xy 80.01 49.53) (xy 80.01 52.07)))
+    (arrow1a (pts (xy 80.01 52.07) (xy 79.423579 50.943496)))
+    (arrow1b (pts (xy 80.01 52.07) (xy 80.596421 50.943496)))
+    (arrow2a (pts (xy 80.01 49.53) (xy 79.423579 50.656504)))
+    (arrow2b (pts (xy 80.01 49.53) (xy 80.596421 50.656504)))
+  )
+  (dimension 2.54 (width 0.15) (layer Dwgs.User)
+    (gr_text "2.540 mm" (at 74.93 45.69) (layer Dwgs.User)
+      (effects (font (size 1 1) (thickness 0.15)))
+    )
+    (feature1 (pts (xy 76.2 48.26) (xy 76.2 46.403579)))
+    (feature2 (pts (xy 73.66 48.26) (xy 73.66 46.403579)))
+    (crossbar (pts (xy 73.66 46.99) (xy 76.2 46.99)))
+    (arrow1a (pts (xy 76.2 46.99) (xy 75.073496 47.576421)))
+    (arrow1b (pts (xy 76.2 46.99) (xy 75.073496 46.403579)))
+    (arrow2a (pts (xy 73.66 46.99) (xy 74.786504 47.576421)))
+    (arrow2b (pts (xy 73.66 46.99) (xy 74.786504 46.403579)))
+  )
   (gr_text PMOD (at 48.006 50.8) (layer F.SilkS)
     (effects (font (size 1 1) (thickness 0.15)))
@@
   )
   (dimension 5.08 (width 0.15) (layer Dwgs.User)
-    (gr_text "0.2000 in" (at 45.72 44.293) (layer Dwgs.User)
-      (effects (font (size 1 1) (thickness 0.15)))
-    )
-    (feature1 (pts (xy 48.26 48.133) (xy 48.26 45.006579)))
-    (feature2 (pts (xy 43.18 48.133) (xy 43.18 45.006579)))
-    (crossbar (pts (xy 43.18 45.593) (xy 48.26 45.593)))
-    (arrow1a (pts (xy 48.26 45.593) (xy 47.133496 46.179421)))
-    (arrow1b (pts (xy 48.26 45.593) (xy 47.133496 45.006579)))
-    (arrow2a (pts (xy 43.18 45.593) (xy 44.306504 46.179421)))
-    (arrow2b (pts (xy 43.18 45.593) (xy 44.306504 45.006579)))
+    (gr_text "0.2000 in" (at 45.72 80.421) (layer Dwgs.User)
+      (effects (font (size 1 1) (thickness 0.15)))
+    )
+    (feature1 (pts (xy 48.26 77.724) (xy 48.26 79.707421)))
+    (feature2 (pts (xy 43.18 77.724) (xy 43.18 79.707421)))
+    (crossbar (pts (xy 43.18 79.121) (xy 48.26 79.121)))
+    (arrow1a (pts (xy 48.26 79.121) (xy 47.133496 79.707421)))
+    (arrow1b (pts (xy 48.26 79.121) (xy 47.133496 78.534579)))
+    (arrow2a (pts (xy 43.18 79.121) (xy 44.306504 79.707421)))
+    (arrow2b (pts (xy 43.18 79.121) (xy 44.306504 78.534579)))
   )
   (gr_text "Theremin Sensor PMOD" (at 61.849 52.197) (layer B.SilkS)
@@
   (gr_circle (center 73.66 52.07) (end 75.36 52.07) (layer Edge.Cuts) (width 0.05))
   (dimension 33.02 (width 0.15) (layer Dwgs.User)
-    (gr_text "33.020 mm" (at 59.69 76.23) (layer Dwgs.User)
-      (effects (font (size 1 1) (thickness 0.15)))
-    )
-    (feature1 (pts (xy 76.2 72.39) (xy 76.2 75.516421)))
-    (feature2 (pts (xy 43.18 72.39) (xy 43.18 75.516421)))
-    (crossbar (pts (xy 43.18 74.93) (xy 76.2 74.93)))
-    (arrow1a (pts (xy 76.2 74.93) (xy 75.073496 75.516421)))
-    (arrow1b (pts (xy 76.2 74.93) (xy 75.073496 74.343579)))
-    (arrow2a (pts (xy 43.18 74.93) (xy 44.306504 75.516421)))
-    (arrow2b (pts (xy 43.18 74.93) (xy 44.306504 74.343579)))
+    (gr_text "33.020 mm" (at 59.69 75.595) (layer Dwgs.User)
+      (effects (font (size 1 1) (thickness 0.15)))
+    )
+    (feature1 (pts (xy 76.2 72.771) (xy 76.2 74.881421)))
+    (feature2 (pts (xy 43.18 72.771) (xy 43.18 74.881421)))
+    (crossbar (pts (xy 43.18 74.295) (xy 76.2 74.295)))
+    (arrow1a (pts (xy 76.2 74.295) (xy 75.073496 74.881421)))
+    (arrow1b (pts (xy 76.2 74.295) (xy 75.073496 73.708579)))
+    (arrow2a (pts (xy 43.18 74.295) (xy 44.306504 74.881421)))
+    (arrow2b (pts (xy 43.18 74.295) (xy 44.306504 73.708579)))
   )
   (gr_line (start 43.18 49.53) (end 76.2 49.53) (layer Edge.Cuts) (width 0.05))
