File: coratheremin/kicad/theremin_z7_lite_main_board/theremin_z7_lite_main_board.kicad_pcb (KiCad board)
At the start: 2 copper layers, 120 x 80 mm, 83 parts, among them J1 GPIO1, J10 EXPR_PED1, J11 EXPR_PED2, J12 +5V Input, J13 LINE_IN_EXT, J14 LINE_OUT_EXT, J15 HP_EXT, J16 POTS, J17 PMOD3, J18 Conn_01x08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

Commit message: controls board pcb
Parts:
- added J20: Ground, Connector_PinHeader_2.54mm:PinHeader_1x01_P2.54mm_Vertical, F.Cu at (142.0, 94.7)
Other:
- board text added: "+"
- board text added: "+5V DC In"
- board text added: "3.3"
- board text added: "39"
- board text added: "40"
- board text added: "B0"
- board text added: "B1"
- board text added: "B2"
- board text added: "B3"
- board text added: "B4"
- board text added: "B5"
- board text added: "B6"
- board text added: "B7"
- board text added: "DCLK"
- board text added: "DE"
- board text added: "Encoders"
- board text added: "Expr Ped 1"
- board text added: "Expr Ped 2"
- board text added: "G0"
- board text added: "G2"
- board text added: "G3"
- board text added: "G4"
- board text added: "G5"
- board text added: "G6"
- board text added: "G7"
- board text added: "GPIO1"
- board text added: "GPIO2"
- board text added: "Ground"
- board text added: "HSYNC"
- board text added: "Line In"
- board text added: "Line Out"
- board text added: "N/C"
- board text added: "PMOD1 (Vol sensor)"
- board text added: "PMOD2 (Pitch sensor)"
- board text added: "PMOD3 (Misc)"
- board text added: "PWM"
- board text added: "Phones"
- board text added: "Pots"
- board text added: "R0"
- board text added: "R1"
- board text added: "R2"
- board text added: "R3"
- board text added: "R4"
- board text added: "R5"
- board text added: "R6"
- board text added: "R7"
- board text added: "S/PDIF Out"
- board text added: "T_BUSY"
- board text added: "T_IRQ"
- board text added: "T_MISO"
- board text added: "T_MOSI"
- board text added: "T_SCK"
- board text added: "T_SEL"
- board text added: "VSYNC"

Commit message: pcbs updated, jlcpcb prod rev 0.1, gerber files
Parts:
- moved F1 4.17 mm to (138.6, 28.6)
- moved D1 2.10 mm to (139.3, 24.1), turned to 180 degrees
Routing:
- net +5V: track 365.1 -> 368.9 mm
- net Net-(D1-Pad1): track 4.07 -> 5.07 mm
