File: coratheremin/kicad/theremin_z7_lite_main_board/theremin_z7_lite_main_board.sch (KiCad schematic (older format))
At the start: 83 parts, among them J1 GPIO1, J10 EXPR_PED1, J11 EXPR_PED2, J12 +5V Input, J13 LINE_IN_EXT, J14 LINE_OUT_EXT, J15 HP_EXT, J16 POTS, J17 PMOD3, J18 Conn_01x08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

Commit message: controls board pcb
Parts:
- added J20: Ground, Connector_PinHeader_2.54mm:PinHeader_1x01_P2.54mm_Vertical, symbol Connector_Generic:Conn_01x01
Connections:
- net GND: now also J20.1 (Pin_1)
Other:
- moved on the sheet: C1, C2, C22, C23, C24, C25, C26, C27, C28, C29, C3, C30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

Commit message: pcbs updated, jlcpcb prod rev 0.1, gerber files
Other:
- note added: "Z7 Lite based FPGA theremin main board"
- moved on the sheet: C37, U5
Changed lines of the file:
@@
 L plt133t10w:PLT133T10W U5
 U 1 1 60A399D2
-P 14900 7000
-F 0 "U5" H 15078 6871 50  0000 L CNN
-F 1 "PLT133T10W" H 15078 6780 50  0000 L CNN
-F 2 "Theremin:PLT133T10W" H 14900 7050 50  0001 C CNN
-F 3 "" H 14900 7050 50  0001 C CNN
-	1    14900 7000
+P 6100 4350
+F 0 "U5" H 6278 4221 50  0000 L CNN
+F 1 "PLT133T10W" H 6278 4130 50  0000 L CNN
+F 2 "Theremin:PLT133T10W" H 6100 4400 50  0001 C CNN
+F 3 "" H 6100 4400 50  0001 C CNN
+	1    6100 4350
 	1    0    0    -1
 $EndComp
@@
 	4800 8850 4900 8950
 Entry Wire Line
-	2850 8650 2950 8750
-Entry Wire Line
-	2850 8750 2950 8850
-Wire Wire Line
-	2950 8750 3650 8750
-Wire Wire Line
-	2950 8850 3650 8850
+	2450 8650 2550 8750
+Entry Wire Line
+	2450 8750 2550 8850
+Wire Wire Line
+	2550 8750 3650 8750
+Wire Wire Line
+	2550 8850 3650 8850
 Wire Wire Line
 	4150 8750 4800 8750
@@
 	4800 9900 4900 10000
 Entry Wire Line
-	2850 9800 2950 9900
-Entry Wire Line
-	2850 9700 2950 9800
-Wire Wire Line
-	2950 9800 3650 9800
-Wire Wire Line
-	2950 9900 3650 9900
+	2450 9800 2550 9900
+Entry Wire Line
+	2450 9700 2550 9800
+Wire Wire Line
+	2550 9800 3650 9800
+Wire Wire Line
+	2550 9900 3650 9900
 Wire Wire Line
 	4150 9900 4800 9900
@@
 L Device:C C37
 U 1 1 62D9F3C2
-P 14350 7450
-F 0 "C37" H 14465 7496 50  0000 L CNN
-F 1 "0.1uF" H 14465 7405 50  0000 L CNN
-F 2 "Capacitor_SMD:C_0805_2012Metric" H 14388 7300 50  0001 C CNN
-F 3 "~" H 14350 7450 50  0001 C CNN
-	1    14350 7450
-	1    0    0    -1
-$EndComp
-Wire Wire Line
-	14700 7200 14350 7200
-Wire Wire Line
-	14350 7200 14350 7300
-Wire Wire Line
-	14700 7300 14700 7700
-Wire Wire Line
-	14700 7700 14350 7700
-Wire Wire Line
-	14350 7700 14350 7600
-Entry Wire Line
-	13700 7000 13800 7100
+P 5550 4800
+F 0 "C37" H 5665 4846 50  0000 L CNN
+F 1 "0.1uF" H 5665 4755 50  0000 L CNN
+F 2 "Capacitor_SMD:C_0805_2012Metric" H 5588 4650 50  0001 C CNN
+F 3 "~" H 5550 4800 50  0001 C CNN
+	1    5550 4800
+	1    0    0    -1
+$EndComp
+Wire Wire Line
+	5900 4550 5550 4550
+Wire Wire Line
+	5550 4550 5550 4650
+Wire Wire Line
+	5900 4650 5900 5050
+Wire Wire Line
+	5900 5050 5550 5050
+Wire Wire Line
+	5550 5050 5550 4950
+Entry Wire Line
+	4900 4350 5000 4450
 $Comp
 L power:+3.3V #PWR0114
 U 1 1 62E2B711
-P 14250 7200
-F 0 "#PWR0114" H 14250 7050 50  0001 C CNN
-F 1 "+3.3V" V 14265 7328 50  0000 L CNN
-F 2 "" H 14250 7200 50  0001 C CNN
-F 3 "" H 14250 7200 50  0001 C CNN
-	1    14250 7200
+P 5450 4550
+F 0 "#PWR0114" H 5450 4400 50  0001 C CNN
+F 1 "+3.3V" V 5465 4678 50  0000 L CNN
+F 2 "" H 5450 4550 50  0001 C CNN
+F 3 "" H 5450 4550 50  0001 C CNN
+	1    5450 4550
 	0    -1   -1   0
 $EndComp
@@
 L power:GND #PWR0115
 U 1 1 62E2C263
-P 14700 7750
-F 0 "#PWR0115" H 14700 7500 50  0001 C CNN
-F 1 "GND" H 14705 7577 50  0000 C CNN
-F 2 "" H 14700 7750 50  0001 C CNN
-F 3 "" H 14700 7750 50  0001 C CNN
-	1    14700 7750
-	1    0    0    -1
-$EndComp
-Wire Wire Line
-	14700 7700 14700 7750
-Connection ~ 14700 7700
-Wire Wire Line
-	14700 7100 13800 7100
-Wire Wire Line
-	14250 7200 14350 7200
-Connection ~ 14350 7200
-Text Label 13900 7100 0    50   ~ 0
+P 5900 5100
+F 0 "#PWR0115" H 5900 4850 50  0001 C CNN
+F 1 "GND" H 5905 4927 50  0000 C CNN
+F 2 "" H 5900 5100 50  0001 C CNN
+F 3 "" H 5900 5100 50  0001 C CNN
+	1    5900 5100
+	1    0    0    -1
+$EndComp
+Wire Wire Line
+	5900 5050 5900 5100
+Connection ~ 5900 5050
+Wire Wire Line
+	5900 4450 5000 4450
+Wire Wire Line
+	5450 4550 5550 4550
+Connection ~ 5550 4550
+Text Label 5100 4450 0    50   ~ 0
 SPDIF_OUT
 Text Label 3200 1650 0    50   ~ 0
@@
 	8150 900  8250 1000
 Wire Bus Line
-	2850 8250 3050 8250
+	2450 8250 3050 8250
 Entry Bus Bus
 	6050 6550 6150 6650
@@
 Wire Bus Line
 	10150 3450 10150 3750
+Text Notes 900  700  0    118  ~ 0
+Z7 Lite based FPGA theremin main board
 Wire Bus Line
 	5000 6550 9900 6550
@@
 	9250 650  15500 650
 Wire Bus Line
-	2850 8250 2850 9900
+	2450 8250 2450 9900
 Wire Bus Line
 	9900 6550 9900 8500
